File: SIGMAGE/SIGMAGE.kicad_pcb (KiCad board)
At the start: 2 copper layers, 100 x 90 mm, 116 parts, among them J1 UJ31CHG2SMTTR, J10 TSW10607GS, J14 HTSW10807GD, J15 HTSW10807GD, J16 HTSW10807GD, J17 HTSW10807GD, J18 HTSW10107GD, J19 HTSW10107GD, J2 SJ63073E, J3 SJ63073E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

Commit message: Almost finished tha board
Parts:
- moved C24 1.12 mm to (127.5, 104.8), turned to 90 degrees
- moved C1 0.75 mm to (147.8, 143.5), turned to 180 degrees
- moved C4 0.75 mm to (166.2, 143.5), turned to 180 degrees
Routing:
- net +5V: track 65.6 -> 212.4 mm, vias 2 -> 5
- net +2V5: track 66.8 -> 175.5 mm, vias 0 -> 5
- net +3V3: track 244.3 -> 329.7 mm, vias 7 -> 23
- net PHY_NRST: track 45.8 -> 50.0 mm, vias 2 -> 4
- net PHY_MDIO: track 29.9 -> 32.8 mm
- net PHY_CRS_DV: track 38.4 -> 41.2 mm
- net PHY_REFCLK: track 30.2 -> 33.0 mm
- net Net-(U8-NRST): track 6.97 -> 9.62 mm, vias 0 -> 1
- net AN2_R: track 18.3 -> 20.1 mm
- net AN1_R: track 18.7 -> 20.5 mm
- net Net-(J6-TD2+): track 26.4 -> 25.7 mm
- added copper zone on F.Cu, net +2V5
