File: SIGMAGE_HW/SIGMAGE/SIGMAGE.kicad_pcb (KiCad board)
At the start: 2 copper layers, 100 x 90 mm, 116 parts, among them J1 UJ31CHG2SMTTR, J10 TSW10607GS, J14 HTSW10807GD, J15 HTSW10807GD, J16 HTSW10807GD, J17 HTSW10807GD, J18 HTSW10107GD, J19 HTSW10107GD, J2 SJ63073E, J3 SJ63073E, J4 SJ63073E, J5 SJ63073E, J6 ARJM11D7502ABEW2, J7 TSW10607GS, J8 TSW10607GS, J9 TSW10607GS, U1 MAX8902BATA/V+T, U2 MAX8902BATA/V+T, U4 OPA1612AIDRGR, U5 PCM1803ADB, U6 OPA1612AIDRGR, U7 PCM1803ADB, U8 STM32F407VGTx, U9 LAN8720ACP, X1 STDCSU18M, X2 STDCSK425M

Commit message: finishing up
Parts:
- removed C14, C15: 100n, Capacitor_SMD:C_0603_1608Metric
- removed D1, D2: LED, LED_SMD:LED_0603_1608Metric
- removed J14, J15, J16, J17: HTSW10807GD, SIGMAGE:HTSW10807GD
- removed J8: TSW10607GS, SIGMAGE:TSW10607GS
- removed R3: 130, Resistor_SMD:R_0603_1608Metric
- removed R6: 50, Resistor_SMD:R_0603_1608Metric
- removed X2: STDCSK425M, SIGMAGE:STDCSK425M
- added C100: 100n, Capacitor_SMD:C_0603_1608Metric, F.Cu at (337.3, 135.9)
- added C101: 100n, Capacitor_SMD:C_0603_1608Metric, F.Cu at (337.3, 138.4)
- added C102: 10u, Capacitor_SMD:C_0603_1608Metric, F.Cu at (337.3, 140.9)
- added C103: 100n, Capacitor_SMD:C_0603_1608Metric, F.Cu at (337.3, 143.4)
- added C104: 100n, Capacitor_SMD:C_0603_1608Metric, F.Cu at (337.3, 145.9)
- added C105: 10u, Capacitor_SMD:C_0603_1608Metric, F.Cu at (341.3, 130.9)
- added C106: 100n, Capacitor_SMD:C_0603_1608Metric, F.Cu at (341.3, 133.4)
- added C107: 100n, Capacitor_SMD:C_0603_1608Metric, F.Cu at (341.3, 135.9)
- added C108: 10u, Capacitor_SMD:C_0603_1608Metric, F.Cu at (341.3, 138.4)
- added C109: 100n, Capacitor_SMD:C_0603_1608Metric, F.Cu at (341.3, 140.9)
- added C110: 100n, Capacitor_SMD:C_0603_1608Metric, F.Cu at (341.3, 143.4)
- added C111: 10u, Capacitor_SMD:C_0603_1608Metric, F.Cu at (341.3, 145.9)
- added C112: 18p, Capacitor_SMD:C_0603_1608Metric, F.Cu at (475.3, 167.0)
- added C113: 18p, Capacitor_SMD:C_0603_1608Metric, F.Cu at (475.3, 169.6)
- added C114: 2.2p, Capacitor_SMD:C_0603_1608Metric, F.Cu at (475.3, 172.1)
- added C115: 2.2p, Capacitor_SMD:C_0603_1608Metric, F.Cu at (475.3, 174.6)
- added C116: 100n, Capacitor_SMD:C_0603_1608Metric, F.Cu at (475.3, 177.1)
- added C117: 100n, Capacitor_SMD:C_0603_1608Metric, F.Cu at (475.3, 179.6)
- added C118: 100n, Capacitor_SMD:C_0603_1608Metric, F.Cu at (479.3, 167.0)
- added C119: 100n, Capacitor_SMD:C_0603_1608Metric, F.Cu at (479.3, 169.6)
- added C120: 100n, Capacitor_SMD:C_0603_1608Metric, F.Cu at (479.3, 172.1)
- added C121: 100n, Capacitor_SMD:C_0603_1608Metric, F.Cu at (479.3, 174.6)
- added C122: 100n, Capacitor_SMD:C_0603_1608Metric, F.Cu at (479.3, 177.1)
- added C123: 100n, Capacitor_SMD:C_0603_1608Metric, F.Cu at (479.3, 179.6)
- added C124: 10u, Capacitor_SMD:C_0603_1608Metric, F.Cu at (483.3, 167.0)
- added C125: 100n, Capacitor_SMD:C_1206_3216Metric, F.Cu at (372.0, 74.8)
- added C126: 10u, Capacitor_SMD:C_1206_3216Metric, F.Cu at (372.0, 78.2)
- added C127: 1u, Capacitor_SMD:C_1206_3216Metric, F.Cu at (372.0, 81.5)
- added C128: 1u, Capacitor_SMD:C_1206_3216Metric, F.Cu at (372.0, 84.9)
- added C129: 1n, Capacitor_SMD:C_1206_3216Metric, F.Cu at (372.0, 88.2)
- added C130: 1n, Capacitor_SMD:C_1206_3216Metric, F.Cu at (372.0, 91.6)
- added C131: 1u, Capacitor_SMD:C_1206_3216Metric, F.Cu at (372.0, 94.9)
- added C132: 1u, Capacitor_SMD:C_1206_3216Metric, F.Cu at (372.0, 98.3)
- added C133: 1n, Capacitor_SMD:C_1206_3216Metric, F.Cu at (377.7, 71.5)
- added C134: 1n, Capacitor_SMD:C_1206_3216Metric, F.Cu at (377.7, 74.8)
- added C135: 100n, Capacitor_SMD:C_1206_3216Metric, F.Cu at (377.7, 78.2)
- added C136: 100n, Capacitor_SMD:C_1206_3216Metric, F.Cu at (377.7, 81.5)
- added C137: 100n, Capacitor_SMD:C_1206_3216Metric, F.Cu at (377.7, 84.9)
- added C138: 100n, Capacitor_SMD:C_1206_3216Metric, F.Cu at (377.7, 88.2)
- added C139: 100n, Capacitor_SMD:C_1206_3216Metric, F.Cu at (377.7, 91.6)
- added C140: 100n, Capacitor_SMD:C_1206_3216Metric, F.Cu at (377.7, 94.9)
- added C141: 100n, Capacitor_SMD:C_1206_3216Metric, F.Cu at (377.7, 98.3)
- added C142: 100n, Capacitor_SMD:C_1206_3216Metric, F.Cu at (383.3, 71.5)
- added C143: 100n, Capacitor_SMD:C_0603_1608Metric, F.Cu at (375.7, 101.2)
- added C144: 100n, Capacitor_SMD:C_0603_1608Metric, F.Cu at (375.7, 103.7)
- added C145: 10u, Capacitor_SMD:C_0603_1608Metric, F.Cu at (434.5, 75.0)
- added C146: 10u, Capacitor_SMD:C_0603_1608Metric, F.Cu at (434.5, 77.5)
- added C147: 10u, Capacitor_SMD:C_0603_1608Metric, F.Cu at (434.5, 80.0)
- added C148: 10u, Capacitor_SMD:C_0603_1608Metric, F.Cu at (434.5, 82.5)
- added C149: 100n, Capacitor_SMD:C_0603_1608Metric, F.Cu at (434.5, 85.0)
- added C150: 100n, Capacitor_SMD:C_0603_1608Metric, F.Cu at (434.5, 87.5)
- added C151: 100n, Capacitor_SMD:C_0603_1608Metric, F.Cu at (434.5, 90.1)
- added C152: 100n, Capacitor_SMD:C_0603_1608Metric, F.Cu at (434.5, 92.6)
- added C153: 10u, Capacitor_SMD:C_0603_1608Metric, F.Cu at (434.5, 95.1)
- added C154: 10u, Capacitor_SMD:C_0603_1608Metric, F.Cu at (438.5, 70.0)
- added C155: 10u, Capacitor_SMD:C_0603_1608Metric, F.Cu at (438.5, 72.5)
- added C156: 10u, Capacitor_SMD:C_0603_1608Metric, F.Cu at (438.5, 75.0)
- added C157: 100n, Capacitor_SMD:C_0603_1608Metric, F.Cu at (438.5, 77.5)
- added C158: 100n, Capacitor_SMD:C_0603_1608Metric, F.Cu at (438.5, 80.0)
- added C159: 100n, Capacitor_SMD:C_0603_1608Metric, F.Cu at (438.5, 82.5)
- added C160: 100n, Capacitor_SMD:C_0603_1608Metric, F.Cu at (438.5, 85.0)
- added C161: 2200n, Capacitor_SMD:C_0603_1608Metric, F.Cu at (438.5, 87.5)
- added C162: 2200n, Capacitor_SMD:C_0603_1608Metric, F.Cu at (438.5, 90.1)
- added C163: 2200n, Capacitor_SMD:C_0603_1608Metric, F.Cu at (438.5, 92.6)
- added C164: 2200n, Capacitor_SMD:C_0603_1608Metric, F.Cu at (438.5, 95.1)
- added C165: 1u, Capacitor_SMD:C_1206_3216Metric, F.Cu at (427.3, 50.3)
- added C166: 1u, Capacitor_SMD:C_1206_3216Metric, F.Cu at (427.3, 53.6)
- added C167: 1u, Capacitor_SMD:C_1206_3216Metric, F.Cu at (427.3, 57.0)
- added C168: 1u, Capacitor_SMD:C_1206_3216Metric, F.Cu at (427.3, 60.3)
- added C169: 1n, Capacitor_SMD:C_0603_1608Metric, F.Cu at (442.5, 70.0)
- added C170: 1n, Capacitor_SMD:C_0603_1608Metric, F.Cu at (442.5, 72.5)
- added C171: 1n, Capacitor_SMD:C_0603_1608Metric, F.Cu at (442.5, 75.0)
- added C172: 1n, Capacitor_SMD:C_0603_1608Metric, F.Cu at (442.5, 77.5)
- added C173: 100n, Capacitor_SMD:C_1206_3216Metric, F.Cu at (383.3, 74.8)
- added C174: 10u, Capacitor_SMD:C_1206_3216Metric, F.Cu at (383.3, 78.2)
- added C175: 100n, Capacitor_SMD:C_1206_3216Metric, F.Cu at (383.3, 81.5)
- added C176: 10u, Capacitor_SMD:C_1206_3216Metric, F.Cu at (383.3, 84.9)
- added C177: 100n, Capacitor_SMD:C_1206_3216Metric, F.Cu at (427.3, 63.7)
- added C178: 10u, Capacitor_SMD:C_1206_3216Metric, F.Cu at (427.3, 67.0)
- added C58: 10u, Capacitor_SMD:C_0603_1608Metric, F.Cu at (426.4, 70.0)
- added C59: 100n, Capacitor_SMD:C_0603_1608Metric, F.Cu at (426.4, 72.5)
- added C60: 10u, Capacitor_SMD:C_0603_1608Metric, F.Cu at (426.4, 75.0)
- added C61: 100n, Capacitor_SMD:C_0603_1608Metric, F.Cu at (426.4, 77.5)
- added C62: 1u, Capacitor_SMD:C_1206_3216Metric, F.Cu at (427.3, 36.9)
- added C63: 1u, Capacitor_SMD:C_1206_3216Metric, F.Cu at (427.3, 40.2)
- added C64: 2200n, Capacitor_SMD:C_0603_1608Metric, F.Cu at (426.4, 80.0)
- added C65: 2200n, Capacitor_SMD:C_0603_1608Metric, F.Cu at (426.4, 82.5)
- added C66: 10u, Capacitor_SMD:C_0603_1608Metric, F.Cu at (426.4, 85.0)
- added C67: 100n, Capacitor_SMD:C_0603_1608Metric, F.Cu at (426.4, 87.5)
- added C68: 10u, Capacitor_SMD:C_0603_1608Metric, F.Cu at (426.4, 90.1)
- added C69: 100n, Capacitor_SMD:C_0603_1608Metric, F.Cu at (426.4, 92.6)
- added C7: 10u, Capacitor_SMD:C_0603_1608Metric, F.Cu at (365.7, 145.9)
- added C70: 1n, Capacitor_SMD:C_0603_1608Metric, F.Cu at (426.4, 95.1)
- added C71: 1n, Capacitor_SMD:C_0603_1608Metric, F.Cu at (430.4, 70.0)
- added C72: 10u, Capacitor_SMD:C_0603_1608Metric, F.Cu at (430.4, 72.5)
- added C73: 10u, Capacitor_SMD:C_0603_1608Metric, F.Cu at (430.4, 75.0)
- added C74: 100n, Capacitor_SMD:C_0603_1608Metric, F.Cu at (430.4, 77.5)
- added C75: 100n, Capacitor_SMD:C_0603_1608Metric, F.Cu at (430.4, 80.0)
- added C76: 10u, Capacitor_SMD:C_0603_1608Metric, F.Cu at (430.4, 82.5)
- added C77: 10u, Capacitor_SMD:C_0603_1608Metric, F.Cu at (430.4, 85.0)
- added C78: 100n, Capacitor_SMD:C_0603_1608Metric, F.Cu at (430.4, 87.5)
- added C79: 100n, Capacitor_SMD:C_0603_1608Metric, F.Cu at (430.4, 90.1)
- added C8: 100n, Capacitor_SMD:C_0603_1608Metric, F.Cu at (365.7, 148.4)
- added C80: 2200n, Capacitor_SMD:C_0603_1608Metric, F.Cu at (430.4, 92.6)
- added C81: 2200n, Capacitor_SMD:C_0603_1608Metric, F.Cu at (430.4, 95.1)
- added C82: 1u, Capacitor_SMD:C_1206_3216Metric, F.Cu at (427.3, 43.6)
- added C83: 1u, Capacitor_SMD:C_1206_3216Metric, F.Cu at (427.3, 46.9)
- added C84: 1n, Capacitor_SMD:C_0603_1608Metric, F.Cu at (434.5, 70.0)
- added C85: 1n, Capacitor_SMD:C_0603_1608Metric, F.Cu at (434.5, 72.5)
- added C86: 1u, Capacitor_SMD:C_0603_1608Metric, F.Cu at (369.7, 148.4)
- added C87: 1u, Capacitor_SMD:C_0603_1608Metric, F.Cu at (369.7, 151.0)
- added C88: 100n, Capacitor_SMD:C_1206_3216Metric, F.Cu at (476.1, 187.6)
- added C89: 100n, Capacitor_SMD:C_1206_3216Metric, F.Cu at (366.4, 98.3)
- added C9: 3300p, Capacitor_SMD:C_0603_1608Metric, F.Cu at (365.7, 151.0)
- added C90: 10u, Capacitor_SMD:C_1206_3216Metric, F.Cu at (372.0, 71.5)
- added C91: 100n, Capacitor_SMD:C_0603_1608Metric, F.Cu at (333.2, 130.9)
- added C92: 100n, Capacitor_SMD:C_0603_1608Metric, F.Cu at (333.2, 133.4)
- added C93: 10u, Capacitor_SMD:C_0603_1608Metric, F.Cu at (333.2, 135.9)
- added C94: 100n, Capacitor_SMD:C_0603_1608Metric, F.Cu at (333.2, 138.4)
- added C95: 100n, Capacitor_SMD:C_0603_1608Metric, F.Cu at (333.2, 140.9)
- added C96: 10u, Capacitor_SMD:C_0603_1608Metric, F.Cu at (333.2, 143.4)
- added C97: 100n, Capacitor_SMD:C_0603_1608Metric, F.Cu at (333.2, 145.9)
- added C98: 100n, Capacitor_SMD:C_0603_1608Metric, F.Cu at (337.3, 130.9)
- added C99: 10u, Capacitor_SMD:C_0603_1608Metric, F.Cu at (337.3, 133.4)
- added CR1: 7M12MAAJT, SIGMAGE:7M12MAAJT, F.Cu at (487.2, 159.9)
- added D10: LED, LED_SMD:LED_0603_1608Metric, F.Cu at (390.2, 143.9)
- added D100: LED, LED_SMD:LED_0603_1608Metric, F.Cu at (406.4, 169.8)
- added D101: LED, LED_SMD:LED_0603_1608Metric, F.Cu at (406.4, 172.4)
- added D102: LED, LED_SMD:LED_0603_1608Metric, F.Cu at (406.4, 174.9)
- added D103: LED, LED_SMD:LED_0603_1608Metric, F.Cu at (406.4, 177.5)
- added D104: LED, LED_SMD:LED_0603_1608Metric, F.Cu at (406.4, 180.1)
- added D105: LED, LED_SMD:LED_0603_1608Metric, F.Cu at (410.4, 130.9)
- added D106: LED, LED_SMD:LED_0603_1608Metric, F.Cu at (410.4, 133.5)
- added D107: LED, LED_SMD:LED_0603_1608Metric, F.Cu at (410.4, 136.1)
- added D108: LED, LED_SMD:LED_0603_1608Metric, F.Cu at (410.4, 138.7)
- added D109: LED, LED_SMD:LED_0603_1608Metric, F.Cu at (410.4, 141.3)
- added D11: LED, LED_SMD:LED_0603_1608Metric, F.Cu at (390.2, 146.5)
- added D110: LED, LED_SMD:LED_0603_1608Metric, F.Cu at (410.4, 143.9)
- added D111: LED, LED_SMD:LED_0603_1608Metric, F.Cu at (410.4, 146.5)
- added D112: LED, LED_SMD:LED_0603_1608Metric, F.Cu at (410.4, 149.0)
- added D113: LED, LED_SMD:LED_0603_1608Metric, F.Cu at (410.4, 151.6)
- added D114: LED, LED_SMD:LED_0603_1608Metric, F.Cu at (410.4, 154.2)
- added D115: LED, LED_SMD:LED_0603_1608Metric, F.Cu at (410.4, 156.8)
- added D116: LED, LED_SMD:LED_0603_1608Metric, F.Cu at (410.4, 159.4)
- added D117: LED, LED_SMD:LED_0603_1608Metric, F.Cu at (410.4, 162.0)
- added D118: LED, LED_SMD:LED_0603_1608Metric, F.Cu at (410.4, 164.6)
- added D119: LED, LED_SMD:LED_0603_1608Metric, F.Cu at (410.4, 167.2)
- added D12: LED, LED_SMD:LED_0603_1608Metric, F.Cu at (390.2, 149.0)
- added D120: LED, LED_SMD:LED_0603_1608Metric, F.Cu at (410.4, 169.8)
- added D121: LED, LED_SMD:LED_0603_1608Metric, F.Cu at (410.4, 172.4)
- added D122: LED, LED_SMD:LED_0603_1608Metric, F.Cu at (410.4, 174.9)
- added D123: LED, LED_SMD:LED_0603_1608Metric, F.Cu at (410.4, 177.5)
- added D124: LED, LED_SMD:LED_0603_1608Metric, F.Cu at (410.4, 180.1)
- added D125: LED, LED_SMD:LED_0603_1608Metric, F.Cu at (414.5, 130.9)
- added D126: LED, LED_SMD:LED_0603_1608Metric, F.Cu at (414.5, 133.5)
- added D127: LED, LED_SMD:LED_0603_1608Metric, F.Cu at (414.5, 136.1)
- added D128: LED, LED_SMD:LED_0603_1608Metric, F.Cu at (414.5, 138.7)
- added D129: LED, LED_SMD:LED_0603_1608Metric, F.Cu at (414.5, 141.3)
- added D13: LED, LED_SMD:LED_0603_1608Metric, F.Cu at (390.2, 151.6)
- added D130: LED, LED_SMD:LED_0603_1608Metric, F.Cu at (414.5, 143.9)
- added D131: LED, LED_SMD:LED_0603_1608Metric, F.Cu at (414.5, 146.5)
- added D132: LED, LED_SMD:LED_0603_1608Metric, F.Cu at (414.5, 149.0)
- added D133: LED, LED_SMD:LED_0603_1608Metric, F.Cu at (414.5, 151.6)
- added D134: LED, LED_SMD:LED_0603_1608Metric, F.Cu at (414.5, 154.2)
- added D135: LED, LED_SMD:LED_0603_1608Metric, F.Cu at (414.5, 156.8)
- added D136: LED, LED_SMD:LED_0603_1608Metric, F.Cu at (414.5, 159.4)
- added D137: LED, LED_SMD:LED_0603_1608Metric, F.Cu at (414.5, 162.0)
- added D138: LED, LED_SMD:LED_0603_1608Metric, F.Cu at (414.5, 164.6)
- added D139: LED, LED_SMD:LED_0603_1608Metric, F.Cu at (414.5, 167.2)
- added D14: LED, LED_SMD:LED_0603_1608Metric, F.Cu at (390.2, 154.2)
- added D140: LED, LED_SMD:LED_0603_1608Metric, F.Cu at (414.5, 169.8)
- added D141: LED, LED_SMD:LED_0603_1608Metric, F.Cu at (414.5, 172.4)
- added D142: LED, LED_SMD:LED_0603_1608Metric, F.Cu at (414.5, 174.9)
- added D143: LED, LED_SMD:LED_0603_1608Metric, F.Cu at (414.5, 177.5)
- added D144: LED, LED_SMD:LED_0603_1608Metric, F.Cu at (414.5, 180.1)
- added D145: LED, LED_SMD:LED_0603_1608Metric, F.Cu at (418.5, 130.9)
- added D146: LED, LED_SMD:LED_0603_1608Metric, F.Cu at (418.5, 133.5)
- added D147: LED, LED_SMD:LED_0603_1608Metric, F.Cu at (418.5, 136.1)
- added D148: LED, LED_SMD:LED_0603_1608Metric, F.Cu at (418.5, 138.7)
- added D149: LED, LED_SMD:LED_0603_1608Metric, F.Cu at (418.5, 141.3)
- added D15: LED, LED_SMD:LED_0603_1608Metric, F.Cu at (390.2, 156.8)
- added D150: LED, LED_SMD:LED_0603_1608Metric, F.Cu at (418.5, 143.9)
- added D151: LED, LED_SMD:LED_0603_1608Metric, F.Cu at (418.5, 146.5)
- added D152: LED, LED_SMD:LED_0603_1608Metric, F.Cu at (418.5, 149.0)
- added D153: LED, LED_SMD:LED_0603_1608Metric, F.Cu at (418.5, 151.6)
- added D154: LED, LED_SMD:LED_0603_1608Metric, F.Cu at (418.5, 154.2)
- added D155: LED, LED_SMD:LED_0603_1608Metric, F.Cu at (418.5, 156.8)
- added D156: LED, LED_SMD:LED_0603_1608Metric, F.Cu at (418.5, 159.4)
- added D157: LED, LED_SMD:LED_0603_1608Metric, F.Cu at (418.5, 162.0)
- added D158: LED, LED_SMD:LED_0603_1608Metric, F.Cu at (418.5, 164.6)
- added D159: LED, LED_SMD:LED_0603_1608Metric, F.Cu at (418.5, 167.2)
- added D16: LED, LED_SMD:LED_0603_1608Metric, F.Cu at (390.2, 159.4)
- added D160: LED, LED_SMD:LED_0603_1608Metric, F.Cu at (418.5, 169.8)
- added D161: LED, LED_SMD:LED_0603_1608Metric, F.Cu at (418.5, 172.4)
- added D162: LED, LED_SMD:LED_0603_1608Metric, F.Cu at (418.5, 174.9)
- added D163: LED, LED_SMD:LED_0603_1608Metric, F.Cu at (418.5, 177.5)
- added D164: LED, LED_SMD:LED_0603_1608Metric, F.Cu at (418.5, 180.1)
- added D165: LED, LED_SMD:LED_0603_1608Metric, F.Cu at (422.6, 130.9)
- added D166: LED, LED_SMD:LED_0603_1608Metric, F.Cu at (422.6, 133.5)
- added D167: LED, LED_SMD:LED_0603_1608Metric, F.Cu at (422.6, 136.1)
- added D168: LED, LED_SMD:LED_0603_1608Metric, F.Cu at (422.6, 138.7)
- added D169: LED, LED_SMD:LED_0603_1608Metric, F.Cu at (422.6, 141.3)
- added D17: LED, LED_SMD:LED_0603_1608Metric, F.Cu at (390.2, 162.0)
- added D170: LED, LED_SMD:LED_0603_1608Metric, F.Cu at (422.6, 143.9)
- added D171: LED, LED_SMD:LED_0603_1608Metric, F.Cu at (422.6, 146.5)
- added D172: LED, LED_SMD:LED_0603_1608Metric, F.Cu at (422.6, 149.0)
- added D173: LED, LED_SMD:LED_0603_1608Metric, F.Cu at (422.6, 151.6)
- added D174: LED, LED_SMD:LED_0603_1608Metric, F.Cu at (422.6, 154.2)
- added D175: LED, LED_SMD:LED_0603_1608Metric, F.Cu at (422.6, 156.8)
- added D176: LED, LED_SMD:LED_0603_1608Metric, F.Cu at (422.6, 159.4)
- added D177: LED, LED_SMD:LED_0603_1608Metric, F.Cu at (422.6, 162.0)
- added D178: LED, LED_SMD:LED_0603_1608Metric, F.Cu at (422.6, 164.6)
- added D179: LED, LED_SMD:LED_0603_1608Metric, F.Cu at (422.6, 167.2)
- added D18: LED, LED_SMD:LED_0603_1608Metric, F.Cu at (390.2, 164.6)
- added D180: LED, LED_SMD:LED_0603_1608Metric, F.Cu at (422.6, 169.8)
- added D181: LED, LED_SMD:LED_0603_1608Metric, F.Cu at (422.6, 172.4)
- added D182: LED, LED_SMD:LED_0603_1608Metric, F.Cu at (422.6, 174.9)
- added D183: LED, LED_SMD:LED_0603_1608Metric, F.Cu at (422.6, 177.5)
- added D184: LED, LED_SMD:LED_0603_1608Metric, F.Cu at (422.6, 180.1)
- added D185: LED, LED_SMD:LED_0603_1608Metric, F.Cu at (426.6, 130.9)
- added D186: LED, LED_SMD:LED_0603_1608Metric, F.Cu at (426.6, 133.5)
- added D187: LED, LED_SMD:LED_0603_1608Metric, F.Cu at (426.6, 136.1)
- added D188: LED, LED_SMD:LED_0603_1608Metric, F.Cu at (426.6, 138.7)
- added D189: LED, LED_SMD:LED_0603_1608Metric, F.Cu at (426.6, 141.3)
- added D19: LED, LED_SMD:LED_0603_1608Metric, F.Cu at (390.2, 167.2)
- added D190: LED, LED_SMD:LED_0603_1608Metric, F.Cu at (426.6, 143.9)
- added D191: LED, LED_SMD:LED_0603_1608Metric, F.Cu at (426.6, 146.5)
- added D192: LED, LED_SMD:LED_0603_1608Metric, F.Cu at (426.6, 149.0)
- added D193: LED, LED_SMD:LED_0603_1608Metric, F.Cu at (426.6, 151.6)
- added D194: LED, LED_SMD:LED_0603_1608Metric, F.Cu at (426.6, 154.2)
- added D195: LED, LED_SMD:LED_0603_1608Metric, F.Cu at (426.6, 156.8)
- added D196: LED, LED_SMD:LED_0603_1608Metric, F.Cu at (426.6, 159.4)
- added D197: LED, LED_SMD:LED_0603_1608Metric, F.Cu at (426.6, 162.0)
- added D198: LED, LED_SMD:LED_0603_1608Metric, F.Cu at (426.6, 164.6)
- added D199: LED, LED_SMD:LED_0603_1608Metric, F.Cu at (426.6, 167.2)
- added D20: LED, LED_SMD:LED_0603_1608Metric, F.Cu at (390.2, 169.8)
- added D200: LED, LED_SMD:LED_0603_1608Metric, F.Cu at (426.6, 169.8)
- added D201: LED, LED_SMD:LED_0603_1608Metric, F.Cu at (426.6, 172.4)
- added D202: LED, LED_SMD:LED_0603_1608Metric, F.Cu at (426.6, 174.9)
- added D203: LED, LED_SMD:LED_0603_1608Metric, F.Cu at (426.6, 177.5)
- added D204: LED, LED_SMD:LED_0603_1608Metric, F.Cu at (426.6, 180.1)
- added D205: LED, LED_SMD:LED_0603_1608Metric, F.Cu at (430.7, 130.9)
- added D206: LED, LED_SMD:LED_0603_1608Metric, F.Cu at (430.7, 133.5)
- added D207: LED, LED_SMD:LED_0603_1608Metric, F.Cu at (430.7, 136.1)
- added D208: LED, LED_SMD:LED_0603_1608Metric, F.Cu at (430.7, 138.7)
- added D209: LED, LED_SMD:LED_0603_1608Metric, F.Cu at (430.7, 141.3)
- added D21: LED, LED_SMD:LED_0603_1608Metric, F.Cu at (390.2, 172.4)
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Connections:
- net AN1_L renamed /ADC/AN1_L
- net AN1_R renamed /ADC/AN1_R
- net AN2_L renamed /ADC/AN2_L
- net AN2_R renamed /ADC/AN2_R
- C1 pad 1: +5V -> VCC_5V
- C11 pad 1: +5V -> VCC_5V
- C13 pad 1: Net-(J3-TIP) -> Net-(J2-RING)
- C19 pad 1: Net-(J5-TIP) -> Net-(J4-RING)
- C20 pad 1: Net-(U4-+INA) -> AVCC_2V5
- C20 pad 2: +2V5 -> Net-(U4-+INA)
- C21 pad 1: Net-(U4-+INB) -> AVCC_2V5
- C21 pad 2: +2V5 -> Net-(U4-+INB)
- C22 pad 1: Net-(U6-+INA) -> AVCC_2V5
- C22 pad 2: +2V5 -> Net-(U6-+INA)
- C23 pad 1: Net-(U6-+INB) -> AVCC_2V5
- C23 pad 2: +2V5 -> Net-(U6-+INB)
- C24 pad 1: GND -> Net-(U7-VREF1)
- C24 pad 2: +3V3 -> GND
- C25 pad 1: Net-(U7-VREF1) -> Net-(U7-VREF2)
- C26 pad 1: GND -> Net-(U18-VREF1)
- C26 pad 2: +5V -> GND
- C27 pad 1: Net-(U7-VREF2) -> Net-(U19-VREF1)
- C28 pad 1: +3V3 -> Net-(U11-VOS)
- C29 pad 1: +3V3 -> VCC_5V
- C30 pad 1: +3V3 -> VCC_5V
- C31 pad 1: +3V3 -> Net-(U12-SS/TR)
- C32 pad 1: +3V3 -> Net-(U12-VOS)
- C33 pad 1: +3V3 -> Net-(U9-VPHY)
- C34 pad 1: +3V3 -> Net-(U9-VPHY)
- C35 pad 1: +3V3 -> Net-(U9-VPLL)
- C36 pad 1: GND -> Net-(U9-VPLL)
- C36 pad 2: +3V3 -> GND
- C37 pad 1: VREF+ -> DVCCFT_1V8
- C38 pad 1: VREF+ -> DVCCFT_1V8
- C39 pad 1: +3V3 -> DVCCFT_1V8
- C4 pad 1: +5V -> VCC_5V
- C40 pad 1: GND -> DVCCFT_1V8
- C40 pad 2: Net-(U8-NRST) -> GND
- C41 pad 1: Net-(U8-PH0) -> DVCC_3V3
- C42 pad 1: Net-(U8-PH1) -> DVCC_3V3
- C43 pad 1: Net-(U8-VCAP_1) -> DVCC_3V3
- C44 pad 1: Net-(U8-VCAP_2) -> DVCC_3V3
- C45 pad 1: GND -> DVCC_3V3
- C45 pad 2: Net-(U9-VDDCR) -> GND
- C46 pad 1: GND -> DVCC_3V3
- C46 pad 2: Net-(U9-VDDCR) -> GND
- C47 pad 1: +3V3 -> Net-(U9-OSCI)
- C48 pad 1: +3V3 -> Net-(U9-OSCO)
- C49 pad 1: +3V3 -> DVCC_1V2
- C50 pad 1: +3V3 -> DVCC_1V2
- C51 pad 1: Net-(U9-XTAL2) -> DVCC_1V2
- C52 pad 1: Net-(U9-XTAL1/CLKIN) -> DVCC_1V2
- C53 pad 1: +3V3 -> DVCC_1V2
- C54 pad 1: +3V3 -> DVCC_1V2
- C55 pad 1: +3V3 -> DVCC_1V2
- FB4 pad 2: +5V -> VCC_5V
- J1 pad A6: unconnected-(J1-DP1-PadA6) -> /USB/USB_DP
- J1 pad A7: unconnected-(J1-DN1-PadA7) -> /USB/USB_DN
- J1 pad B6: unconnected-(J1-DP2-PadB6) -> /USB/USB_DP
- J1 pad B7: unconnected-(J1-DN2-PadB7) -> /USB/USB_DN
- J10 pad 1: JTRST -> GND
- J10 pad 2: JTDO_SWO -> Net-(J10-TIP)
- J10 pad 3: JTDI -> Net-(J10-RING)
- J10 pad 4: JTCK_SWCLK -> unconnected-(J10-SLEEVE_SWITCH-Pad4)
- J10 pad 5: JTMS_SWDIO -> unconnected-(J10-TIP_SWITCH-Pad5)
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Routing:
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- added copper zone on F.Cu, net (none)
- removed copper zone on F.Cu, net +2V5
- removed copper zone on F.Cu, net +3V3
- removed copper zone on F.Cu, net +5V
- removed copper zone on F.Cu, net Net-(D1-A)
- removed copper zone on F.Cu, net Net-(D2-A)
- removed copper zone on F.Cu, net Net-(R2-Pad2)
- removed copper zone on F.Cu, net Net-(R32-Pad1)
- removed copper zone on F.Cu, net Net-(U8-VCAP_1)
- removed copper zone on F.Cu, net Net-(U8-VCAP_2)
- removed copper zone on F.Cu, net Net-(U9-VDDCR)
- removed copper zone on F.Cu, net VREF+
Other:
- board outline removed

Commit message: almost done
Parts:
- removed C17, C24, C25, C26, C27: 100n, Capacitor_SMD:C_0603_1608Metric
- added C14: 10u, Capacitor_SMD:C_0603_1608Metric, F.Cu at (193.2, 169.3)
- added C15: 10n, Capacitor_SMD:C_0603_1608Metric, F.Cu at (193.2, 171.8)
- added C179: 100n, Capacitor_SMD:C_1206_3216Metric, F.Cu at (119.7, 91.8)
- added C180: 100n, Capacitor_SMD:C_1206_3216Metric, F.Cu at (119.7, 95.1)
- added C181: 100n, Capacitor_SMD:C_1206_3216Metric, F.Cu at (119.7, 98.5)
- added C182: 100n, Capacitor_SMD:C_1206_3216Metric, F.Cu at (119.7, 101.8)
- added C183: 100n, Capacitor_SMD:C_1206_3216Metric, F.Cu at (119.7, 105.2)
- added C184: 100n, Capacitor_SMD:C_1206_3216Metric, F.Cu at (119.7, 108.5)
- added C185: 100n, Capacitor_SMD:C_1206_3216Metric, F.Cu at (119.7, 111.9)
- added C186: 100n, Capacitor_SMD:C_1206_3216Metric, F.Cu at (119.7, 115.2)
- added C187: 22u, Capacitor_SMD:C_0603_1608Metric, F.Cu at (201.2, 154.2)
- added C188: 1u, Capacitor_SMD:C_0603_1608Metric, F.Cu at (201.2, 156.8)
- added C189: 1u, Capacitor_SMD:C_0603_1608Metric, F.Cu at (174.0, 213.0)
- added C190: 100n, Capacitor_SMD:C_0603_1608Metric, F.Cu at (174.0, 215.5)
- added C191: 100n, Capacitor_SMD:C_0603_1608Metric, F.Cu at (178.0, 192.9)
- added C192: 22u, Capacitor_SMD:C_0603_1608Metric, F.Cu at (178.0, 195.4)
- added D261: LED, LED_SMD:LED_0603_1608Metric, F.Cu at (186.1, 210.0)
- added D262: LED, LED_SMD:LED_0603_1608Metric, F.Cu at (186.1, 212.6)
- added FB10: 120 @ 100 MHz, Capacitor_SMD:C_0603_1608Metric, F.Cu at (178.0, 197.9)
- added FB8: 500 @ 100 MHz, Capacitor_SMD:C_0603_1608Metric, F.Cu at (201.2, 169.3)
- added FB9: 500 @ 100 MHz, Capacitor_SMD:C_0603_1608Metric, F.Cu at (201.2, 171.8)
- added J26: HTSW10107GD, SIGMAGE:HTSW10107GD, F.Cu at (212.4, 141.2)
- added J27: HTSW10107GD, SIGMAGE:HTSW10107GD, F.Cu at (217.1, 141.2)
- added R117: 10k, Resistor_SMD:R_0603_1608Metric, F.Cu at (134.5, 129.6)
- added R118: 10k, Resistor_SMD:R_0603_1608Metric, F.Cu at (134.5, 132.1)
- added R119: 10k, Resistor_SMD:R_0603_1608Metric, F.Cu at (134.5, 134.6)
- added R120: 10k, Resistor_SMD:R_0603_1608Metric, F.Cu at (138.6, 114.5)
- added R121: 10k, Resistor_SMD:R_0603_1608Metric, F.Cu at (138.6, 117.0)
- added R122: 10k, Resistor_SMD:R_0603_1608Metric, F.Cu at (138.6, 119.5)
- added R123: 10k, Resistor_SMD:R_0603_1608Metric, F.Cu at (138.6, 122.0)
- added R124: 10k, Resistor_SMD:R_0603_1608Metric, F.Cu at (138.6, 124.5)
- added R125: 10k, Resistor_SMD:R_0603_1608Metric, F.Cu at (138.6, 127.0)
- added R126: 10k, Resistor_SMD:R_0603_1608Metric, F.Cu at (138.6, 129.6)
- added R127: 10k, Resistor_SMD:R_0603_1608Metric, F.Cu at (138.6, 132.1)
- added R128: 10k, Resistor_SMD:R_0603_1608Metric, F.Cu at (138.6, 134.6)
- added R129: 10k, Resistor_SMD:R_0603_1608Metric, F.Cu at (142.6, 114.5)
- added R130: 10k, Resistor_SMD:R_0603_1608Metric, F.Cu at (142.6, 117.0)
- added R131: 10k, Resistor_SMD:R_0603_1608Metric, F.Cu at (142.6, 119.5)
- added R132: 10k, Resistor_SMD:R_0603_1608Metric, F.Cu at (142.6, 122.0)
- added R133: 10k, Resistor_SMD:R_0603_1608Metric, F.Cu at (142.6, 124.5)
- added R134: 10k, Resistor_SMD:R_0603_1608Metric, F.Cu at (142.6, 127.0)
- added R135: 10k, Resistor_SMD:R_0603_1608Metric, F.Cu at (142.6, 129.6)
- added R136: 10k, Resistor_SMD:R_0603_1608Metric, F.Cu at (142.6, 132.1)
- added R137: 10k, Resistor_SMD:R_0603_1608Metric, F.Cu at (142.6, 134.6)
- added R138: 10k, Resistor_SMD:R_0603_1608Metric, F.Cu at (146.6, 114.5)
- added R139: 10k, Resistor_SMD:R_0603_1608Metric, F.Cu at (146.6, 117.0)
- added R140: 10k, Resistor_SMD:R_0603_1608Metric, F.Cu at (146.6, 119.5)
- added R141: 10k, Resistor_SMD:R_0603_1608Metric, F.Cu at (146.6, 122.0)
- added R142: 10k, Resistor_SMD:R_0603_1608Metric, F.Cu at (146.6, 124.5)
- added R143: 10k, Resistor_SMD:R_0603_1608Metric, F.Cu at (146.6, 127.0)
- added R144: 10k, Resistor_SMD:R_0603_1608Metric, F.Cu at (146.6, 129.6)
- added R145: 10k, Resistor_SMD:R_0603_1608Metric, F.Cu at (146.6, 132.1)
- added R146: 10k, Resistor_SMD:R_0603_1608Metric, F.Cu at (146.6, 134.6)
- added R147: 10k, Resistor_SMD:R_0603_1608Metric, F.Cu at (178.0, 215.5)
- added R148: 10k, Resistor_SMD:R_0603_1608Metric, F.Cu at (182.0, 192.9)
- added R149: 10k, Resistor_SMD:R_0603_1608Metric, F.Cu at (182.0, 195.4)
- added R150: 650, Resistor_SMD:R_0603_1608Metric, F.Cu at (182.0, 197.9)
- added R151: 10k, Resistor_SMD:R_0603_1608Metric, F.Cu at (182.0, 200.4)
- added R152: 10k, Resistor_SMD:R_0603_1608Metric, F.Cu at (182.0, 202.9)
- added R153: 10k, Resistor_SMD:R_0603_1608Metric, F.Cu at (182.0, 205.4)
- added R154: 60k, Resistor_SMD:R_0603_1608Metric, F.Cu at (209.2, 159.3)
- added R155: 120k, Resistor_SMD:R_0603_1608Metric, F.Cu at (209.2, 161.8)
- added R156: 10k, Resistor_SMD:R_0603_1608Metric, F.Cu at (182.0, 207.9)
- added R3: 440k, Resistor_SMD:R_0603_1608Metric, F.Cu at (205.2, 151.7)
- added R58: 120k, Resistor_SMD:R_0603_1608Metric, F.Cu at (209.2, 154.2)
- added R6: 440k, Resistor_SMD:R_0603_1608Metric, F.Cu at (205.2, 159.3)
- added U31: MAX8902BATA/V+T, SIGMAGE:MAX8902BATAVT, F.Cu at (219.5, 154.9)
- added U32: EC11E183440C, SIGMAGE:EC11E183440C, F.Cu at (187.9, 91.6)
- added U33: EC11E183440C, SIGMAGE:EC11E183440C, F.Cu at (206.7, 91.6)
- added U34: EC11E183440C, SIGMAGE:EC11E183440C, F.Cu at (225.5, 91.6)
- added U35: EC11E183440C, SIGMAGE:EC11E183440C, F.Cu at (131.4, 110.9)
- added U36: EC11E183440C, SIGMAGE:EC11E183440C, F.Cu at (150.2, 110.9)
- added U37: EC11E183440C, SIGMAGE:EC11E183440C, F.Cu at (169.0, 110.9)
- added U38: EC11E183440C, SIGMAGE:EC11E183440C, F.Cu at (187.9, 110.9)
- added U39: EC11E183440C, SIGMAGE:EC11E183440C, F.Cu at (206.7, 110.9)
- added U40: EC11E183440C, SIGMAGE:EC11E183440C, F.Cu at (225.5, 110.9)
- added U41: MMBT2222A, SIGMAGE:MMBT2222A, F.Cu at (190.4, 211.1)
- added U42: TPS62130RGTT, SIGMAGE:TPS62130RGTT, F.Cu at (214.0, 159.1)
- C10, C11: value 2u2 -> 2.2u
- C143: value 100n -> 1u
- C144, C16: value 100n -> 10u
- C177: footprint Capacitor_SMD:C_1206_3216Metric -> Capacitor_SMD:C_0603_1608Metric
- C178: value 10u -> 3300p; footprint Capacitor_SMD:C_1206_3216Metric -> Capacitor_SMD:C_0603_1608Metric
- FB6, FB7: value 500 @ 100 MHz -> 600 @ 100 MHz
- R100, R101, R102, R103, R104, R105, R106, R91, R92, R93, R94, R95, R96, R97, R98, R99: value 1k -> 260
- R111: value 10k -> 650
- R112: value 10k -> 100k
- R12: value 150 -> 1500
- R24: value 60k -> 255k
- U30: value OPA1612AIDRGR -> EC11E183440C; footprint SIGMAGE:OPA1612AIDRGR -> SIGMAGE:EC11E183440C
- moved R73 379.2 mm to (126.5, 129.6)
- moved R75 379.2 mm to (126.5, 134.6)
- moved R74 379.2 mm to (126.5, 132.1)
- moved R79 377.4 mm to (130.5, 122.0)
- moved R80 377.4 mm to (130.5, 124.5)
- moved R81 377.4 mm to (130.5, 127.0)
- moved R82 377.4 mm to (130.5, 129.6)
- moved R84 377.4 mm to (130.5, 134.6)
- moved R83 377.4 mm to (130.5, 132.1)
- moved R85 375.8 mm to (134.5, 114.5)
- moved R86 375.8 mm to (134.5, 117.0)
- moved R87 375.8 mm to (134.5, 119.5)
- moved R88 375.8 mm to (134.5, 122.0)
- moved R89 375.8 mm to (134.5, 124.5)
- moved R90 375.8 mm to (134.5, 127.0)
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Connections:
- net /ADC/AN1_L renamed /ADC/AN_IN1_L
- net /ADC/AN1_R renamed /ADC/AN_IN1_R
- net /ADC/AN2_L renamed /ADC/AN_IN2_L
- net /ADC/AN2_R renamed /ADC/AN_IN2_R
- net /ADC/AN3_L renamed /ADC/AN_IN3_L
- net /ADC/AN3_R renamed /ADC/AN_IN3_R
- net /ADC/AN4_L renamed /ADC/AN_IN4_L
- net /ADC/AN4_R renamed /ADC/AN_IN4_R
- C125 pad 1: VCC_5V -> AVCC_5V
- C126 pad 1: VCC_5V -> AVCC_5V
- C136 pad 1: VCC_5V -> AVCC_5V
- C138 pad 1: VCC_5V -> AVCC_5V
- C141 pad 1: VCC_5V -> AVCC_5V
- C142 pad 1: VCC_5V -> AVCC_5V
- C143 pad 1: Net-(U18-VREF2) -> Net-(C143-Pad1)
- C144 pad 1: Net-(U19-VREF2) -> VCC_5V
- C16 pad 1: Net-(U5-VREF1) -> Net-(U31-OUT)
- C173 pad 1: VCC_5V -> AVCC_5V
- C174 pad 1: VCC_5V -> AVCC_5V
- C175 pad 1: VCC_5V -> AVCC_5V
- C176 pad 1: VCC_5V -> AVCC_5V
- C178 pad 1: VCC_5V -> Net-(U42-SS/TR)
- C89 pad 1: VCC_5V -> AVCC_5V
- C90 pad 1: VCC_5V -> AVCC_5V
- J23 pad 1: DVCC_1V2 -> DVCC_2V5
- R110 pad 2: DVCC_3V3 -> Net-(R110-Pad2)
- R111 pad 1: /FPGA/FPGA_INITN -> Net-(D262-A)
- R112 pad 1: /FPGA/FPGA_PROGRAMN -> Net-(U42-VOS)
- R112 pad 2: DVCC_3V3 -> Net-(U42-PG)
- U10 pad 12: GND -> /DAC/DAC2_SCK
- U16 pad 8: VCC_5V -> AVCC_5V
- U17 pad 8: VCC_5V -> AVCC_5V
- U18 pad 5: VCC_5V -> AVCC_5V
- U19 pad 5: VCC_5V -> AVCC_5V
- U20 pad 12: GND -> /DAC/DAC3_SCK
- U21 pad 12: GND -> /DAC/DAC4_SCK
- U3 pad 12: GND -> /DAC/DAC1_SCK
- U4 pad 8: VCC_5V -> AVCC_5V
- U5 pad 5: VCC_5V -> AVCC_5V
- U6 pad 8: VCC_5V -> AVCC_5V
- U7 pad 5: VCC_5V -> AVCC_5V
- U8 pad G11: unconnected-(U8A-VCCAUX_1-PadG11) -> Net-(U8A-VCCAUX_1)
- U8 pad L7: unconnected-(U8A-VCCAUX_2-PadL7) -> Net-(U8A-VCCAUX_1)
- U8 pad N8: unconnected-(U8F-PB15A-PadN8) -> /FPGA/FPGA_HOLDN
Routing:
- removed copper zone on F.Cu, net (none)
- removed copper zone on B.Cu, net GND
- removed copper zone on F.Cu, net GND
- removed copper zone on F.Cu, net Net-(C56-Pad1)
- removed copper zone on F.Cu, net Net-(C57-Pad1)
- removed copper zone on F.Cu, net Net-(D4-A)
- removed copper zone on F.Cu, net Net-(U1-BYP)
- removed copper zone on F.Cu, net Net-(U1-FB)
- removed copper zone on F.Cu, net Net-(U1-OUT)
- removed copper zone on F.Cu, net Net-(U2-BYP)
- removed copper zone on F.Cu, net Net-(U2-FB)
- removed copper zone on F.Cu, net Net-(U2-OUT)
- removed copper zone on F.Cu, net Net-(U5-VREF1)
- removed copper zone on F.Cu, net Net-(U5-VREF2)
- removed copper zone on F.Cu, net Net-(U7-VREF1)
- removed copper zone on F.Cu, net Net-(U7-VREF2)
- removed copper zone on F.Cu, net VBUS
Other:
- board outline added: 186.6 x 196 mm

Commit message: before sync sheets
Parts:
- added C17: 100n, Capacitor_SMD:C_0603_1608Metric, F.Cu at (161.7, 190.9)
- added C193: 100n, Capacitor_SMD:C_0603_1608Metric, F.Cu at (161.7, 203.4)
- added C194: 100n, Capacitor_SMD:C_0603_1608Metric, F.Cu at (165.7, 190.9)
- added C195: 100n, Capacitor_SMD:C_0603_1608Metric, F.Cu at (165.7, 193.4)
- added C196: 100n, Capacitor_SMD:C_0603_1608Metric, F.Cu at (165.7, 195.9)
- added C197: 100n, Capacitor_SMD:C_0603_1608Metric, F.Cu at (165.7, 198.4)
- added C198: 100n, Capacitor_SMD:C_0603_1608Metric, F.Cu at (165.7, 200.9)
- added C199: 100n, Capacitor_SMD:C_0603_1608Metric, F.Cu at (165.7, 203.4)
- added C24: 100n, Capacitor_SMD:C_0603_1608Metric, F.Cu at (161.7, 193.4)
- added C25: 100n, Capacitor_SMD:C_0603_1608Metric, F.Cu at (161.7, 195.9)
- added C26: 100n, Capacitor_SMD:C_0603_1608Metric, F.Cu at (161.7, 198.4)
- added C27: 100n, Capacitor_SMD:C_0603_1608Metric, F.Cu at (161.7, 200.9)
- added D263: LED, LED_SMD:LED_0603_1608Metric, F.Cu at (193.6, 157.2)
- added D264: LED, LED_SMD:LED_0603_1608Metric, F.Cu at (193.6, 159.8)
- added D265: LED, LED_SMD:LED_0603_1608Metric, F.Cu at (193.6, 162.4)
- added D266: LED, LED_SMD:LED_0603_1608Metric, F.Cu at (193.6, 165.0)
- added D267: LED, LED_SMD:LED_0603_1608Metric, F.Cu at (193.6, 167.6)
- added D268: LED, LED_SMD:LED_0603_1608Metric, F.Cu at (193.6, 170.2)
- added D269: LED, LED_SMD:LED_0603_1608Metric, F.Cu at (197.7, 157.2)
- added D270: LED, LED_SMD:LED_0603_1608Metric, F.Cu at (197.7, 159.8)
- added D271: LED, LED_SMD:LED_0603_1608Metric, F.Cu at (197.7, 162.4)
- added D272: LED, LED_SMD:LED_0603_1608Metric, F.Cu at (197.7, 165.0)
- added D273: LED, LED_SMD:LED_0603_1608Metric, F.Cu at (197.7, 167.6)
- added D274: LED, LED_SMD:LED_0603_1608Metric, F.Cu at (197.7, 170.2)
- added D275: LED, LED_SMD:LED_0603_1608Metric, F.Cu at (201.7, 157.2)
- added D276: LED, LED_SMD:LED_0603_1608Metric, F.Cu at (201.7, 159.8)
- added D277: LED, LED_SMD:LED_0603_1608Metric, F.Cu at (201.7, 162.4)
- added D278: LED, LED_SMD:LED_0603_1608Metric, F.Cu at (201.7, 165.0)
- added J12: DF40C-40DS-0.4V_51, SIGMAGE:DF40C40DS04V51, F.Cu at (237.9, 176.9)
- added J13: DF40C-40DP-0.4V_51, SIGMAGE:DF40C40DP04V51, F.Cu at (251.0, 183.2)
- added J14: DF40C-40DS-0.4V_51, SIGMAGE:DF40C40DS04V51, F.Cu at (237.9, 183.8)
- added J8: DF40C-40DP-0.4V_51, SIGMAGE:DF40C40DP04V51, F.Cu at (251.0, 176.7)
- added R157: 10k, Resistor_SMD:R_0603_1608Metric, F.Cu at (169.7, 190.9)
- added R158: 10k, Resistor_SMD:R_0603_1608Metric, F.Cu at (169.7, 193.4)
- added R159: 10k, Resistor_SMD:R_0603_1608Metric, F.Cu at (169.7, 195.9)
- added R160: 10k, Resistor_SMD:R_0603_1608Metric, F.Cu at (169.7, 198.4)
- added R161: 10k, Resistor_SMD:R_0603_1608Metric, F.Cu at (169.7, 200.9)
- added R162: 10k, Resistor_SMD:R_0603_1608Metric, F.Cu at (169.7, 203.4)
- added R163: 10k, Resistor_SMD:R_0603_1608Metric, F.Cu at (173.7, 190.9)
- added R164: 10k, Resistor_SMD:R_0603_1608Metric, F.Cu at (173.7, 193.4)
- added R165: 10k, Resistor_SMD:R_0603_1608Metric, F.Cu at (173.7, 195.9)
- added R166: 10k, Resistor_SMD:R_0603_1608Metric, F.Cu at (173.7, 198.4)
- added R167: 10k, Resistor_SMD:R_0603_1608Metric, F.Cu at (173.7, 200.9)
- added R168: 10k, Resistor_SMD:R_0603_1608Metric, F.Cu at (173.7, 203.4)
- added R169: 650, Resistor_SMD:R_0603_1608Metric, F.Cu at (197.6, 154.7)
- added R170: 650, Resistor_SMD:R_0603_1608Metric, F.Cu at (201.6, 137.1)
- added R171: 650, Resistor_SMD:R_0603_1608Metric, F.Cu at (201.6, 139.6)
- added R172: 650, Resistor_SMD:R_0603_1608Metric, F.Cu at (201.6, 142.1)
- added R173: 650, Resistor_SMD:R_0603_1608Metric, F.Cu at (201.6, 144.6)
- added R174: 650, Resistor_SMD:R_0603_1608Metric, F.Cu at (201.6, 147.1)
- added R175: 650, Resistor_SMD:R_0603_1608Metric, F.Cu at (201.6, 149.6)
- added R176: 650, Resistor_SMD:R_0603_1608Metric, F.Cu at (201.6, 152.1)
- added R177: 650, Resistor_SMD:R_0603_1608Metric, F.Cu at (201.6, 154.7)
- added R178: 650, Resistor_SMD:R_0603_1608Metric, F.Cu at (205.6, 137.1)
- added R179: 650, Resistor_SMD:R_0603_1608Metric, F.Cu at (205.6, 139.6)
- added R180: 650, Resistor_SMD:R_0603_1608Metric, F.Cu at (205.6, 142.1)
- added R181: 650, Resistor_SMD:R_0603_1608Metric, F.Cu at (205.6, 144.6)
- added R182: 650, Resistor_SMD:R_0603_1608Metric, F.Cu at (205.6, 147.1)
- added R183: 650, Resistor_SMD:R_0603_1608Metric, F.Cu at (205.6, 149.6)
- added R184: 650, Resistor_SMD:R_0603_1608Metric, F.Cu at (205.6, 152.1)
- added R185: 1k, Resistor_SMD:R_0603_1608Metric, F.Cu at (249.9, 218.4)
- added S1: TL2201EEYA, SIGMAGE:TL2201EEYA, F.Cu at (130.7, 195.4)
- added S10: TL2201EEYA, SIGMAGE:TL2201EEYA, F.Cu at (130.7, 231.9)
- added S11: TL2201EEYA, SIGMAGE:TL2201EEYA, F.Cu at (142.3, 231.9)
- added S12: TL2201EEYA, SIGMAGE:TL2201EEYA, F.Cu at (153.9, 231.9)
- added S2: TL2201EEYA, SIGMAGE:TL2201EEYA, F.Cu at (142.3, 195.4)
- added S3: TL2201EEYA, SIGMAGE:TL2201EEYA, F.Cu at (153.9, 195.4)
- added S4: TL2201EEYA, SIGMAGE:TL2201EEYA, F.Cu at (130.7, 207.6)
- added S5: TL2201EEYA, SIGMAGE:TL2201EEYA, F.Cu at (142.3, 207.6)
- added S6: TL2201EEYA, SIGMAGE:TL2201EEYA, F.Cu at (153.9, 207.6)
- added S7: TL2201EEYA, SIGMAGE:TL2201EEYA, F.Cu at (130.7, 219.7)
- added S8: TL2201EEYA, SIGMAGE:TL2201EEYA, F.Cu at (142.3, 219.7)
- added S9: TL2201EEYA, SIGMAGE:TL2201EEYA, F.Cu at (153.9, 219.7)
- R107: value 10k -> 4700
- moved C10 69.5 mm to (193.6, 174.7)
- moved C11 69.5 mm to (193.6, 177.2)
- moved C33 69.5 mm to (193.6, 179.7)
- moved C34 69.5 mm to (193.6, 182.2)
- moved C35 69.5 mm to (193.6, 184.7)
- moved C36 69.5 mm to (193.6, 187.3)
- moved C37 69.5 mm to (193.6, 189.8)
- moved C38 69.5 mm to (193.6, 192.3)
- moved C39 69.5 mm to (197.6, 174.7)
- moved C40 69.5 mm to (197.6, 177.2)
- moved C41 69.5 mm to (197.6, 179.7)
- moved C42 69.5 mm to (197.6, 182.2)
- moved C43 69.5 mm to (197.6, 184.7)
- moved C44 69.5 mm to (197.6, 187.3)
- moved C45 69.5 mm to (197.6, 189.8)
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Connections:
- net /LED/LED_C0 renamed /LED/T_LED_C1
- net /LED/LED_C1 renamed /LED/T_LED_C2
- net /LED/LED_C10 renamed /LED/T_LED_C11
- net /LED/LED_C11 renamed /LED/T_LED_C12
- net /LED/LED_C12 renamed /LED/T_LED_C13
- net /LED/LED_C13 renamed /LED/T_LED_C14
- net /LED/LED_C14 renamed /LED/T_LED_C15
- net /LED/LED_C15 renamed /LED/T_LED_C16
- net /LED/LED_C2 renamed /LED/T_LED_C3
- net /LED/LED_C3 renamed /LED/T_LED_C4
- net /LED/LED_C4 renamed /LED/T_LED_C5
- net /LED/LED_C5 renamed /LED/T_LED_C6
- net /LED/LED_C6 renamed /LED/T_LED_C7
- net /LED/LED_C7 renamed /LED/T_LED_C8
- net /LED/LED_C8 renamed /LED/T_LED_C9
- net /LED/LED_C9 renamed /LED/T_LED_C10
- net /LED/LED_R0 renamed /LED/T_LED_R1
- net /LED/LED_R1 renamed /LED/T_LED_R2
- net /LED/LED_R10 renamed /LED/T_LED_R11
- net /LED/LED_R11 renamed /LED/T_LED_R12
- net /LED/LED_R12 renamed /LED/T_LED_R13
- net /LED/LED_R13 renamed /LED/T_LED_R14
- net /LED/LED_R14 renamed /LED/T_LED_R15
- net /LED/LED_R15 renamed /LED/T_LED_R16
- net /LED/LED_R2 renamed /LED/T_LED_R3
- net /LED/LED_R3 renamed /LED/T_LED_R4
- net /LED/LED_R4 renamed /LED/T_LED_R5
- net /LED/LED_R5 renamed /LED/T_LED_R6
- net /LED/LED_R6 renamed /LED/T_LED_R7
- net /LED/LED_R7 renamed /LED/T_LED_R8
- net /LED/LED_R8 renamed /LED/T_LED_R9
- net /LED/LED_R9 renamed /LED/T_LED_R10
- J5 pad 1: /MCU/MCU_USART1_TX -> DVCC_3V3
- J5 pad 2: /MCU/MCU_USART1_RX -> /MCU/MCU_USART1_TX
- J5 pad 3: unconnected-(J5-Pad3) -> /MCU/MCU_USART1_RX
- J9 pad 1: /FPGA/FPGA_USART1_TX -> DVCC_3V3
- J9 pad 2: /FPGA/FPGA_USART1_RX -> /FPGA/FPGA_USART1_TX
- J9 pad 3: unconnected-(J9-Pad3) -> /FPGA/FPGA_USART1_RX
- U15 pad 1: unconnected-(U15-PE2-Pad1) -> /MCU/ICOM_AUX2
- U15 pad 2: unconnected-(U15-PE3-Pad2) -> /MCU/ICOM_AUX3
- U15 pad 3: unconnected-(U15-PE4-Pad3) -> /MCU/ICOM_AUX4
- U15 pad 38: unconnected-(U15-PE7-Pad38) -> /MCU/ICOM_AUX7
- U15 pad 39: unconnected-(U15-PE8-Pad39) -> /MCU/ICOM_AUX8
- U15 pad 4: unconnected-(U15-PE5-Pad4) -> /MCU/ICOM_AUX5
- U15 pad 40: unconnected-(U15-PE9-Pad40) -> /MCU/ICOM_AUX9
- U15 pad 41: unconnected-(U15-PE10-Pad41) -> /MCU/ICOM_AUX10
- U15 pad 42: unconnected-(U15-PE11-Pad42) -> /MCU/ICOM_AUX11
- U15 pad 43: unconnected-(U15-PE12-Pad43) -> /MCU/ICOM_AUX12
- U15 pad 44: unconnected-(U15-PE13-Pad44) -> /MCU/ICOM_AUX13
- U15 pad 45: unconnected-(U15-PE14-Pad45) -> /MCU/ICOM_AUX14
- U15 pad 46: unconnected-(U15-PE15-Pad46) -> /MCU/ICOM_AUX15
- U15 pad 5: unconnected-(U15-PE6-Pad5) -> /MCU/ICOM_AUX6
- U15 pad 55: /MCU/ICOM_AUX8 -> Net-(D271-A)
- U15 pad 56: /MCU/ICOM_AUX9 -> Net-(D272-A)
- U15 pad 57: /MCU/ICOM_AUX10 -> Net-(D273-A)
- U15 pad 58: /MCU/ICOM_AUX11 -> Net-(D274-A)
- U15 pad 59: /MCU/ICOM_AUX12 -> Net-(D275-A)
- U15 pad 60: /MCU/ICOM_AUX13 -> Net-(D276-A)
- U15 pad 61: /MCU/ICOM_AUX14 -> Net-(D277-A)
- U15 pad 62: /MCU/ICOM_AUX15 -> Net-(D278-A)
- U15 pad 78: unconnected-(U15-PC10-Pad78) -> /MCU/ICOM_USART3_TX
- U15 pad 79: unconnected-(U15-PC11-Pad79) -> /MCU/ICOM_USART3_RX
- U15 pad 81: /MCU/ICOM_AUX0 -> Net-(D263-A)
- U15 pad 82: /MCU/ICOM_AUX1 -> Net-(D264-A)
- U15 pad 83: /MCU/ICOM_AUX2 -> Net-(D265-A)
- U15 pad 84: /MCU/ICOM_AUX3 -> Net-(D266-A)
- U15 pad 85: /MCU/ICOM_AUX4 -> Net-(D267-A)
- U15 pad 86: /MCU/ICOM_AUX5 -> Net-(D268-A)
- U15 pad 87: /MCU/ICOM_AUX6 -> Net-(D269-A)
- U15 pad 88: /MCU/ICOM_AUX7 -> Net-(D270-A)
- U15 pad 97: unconnected-(U15-PE0-Pad97) -> /MCU/ICOM_AUX0
- U15 pad 98: unconnected-(U15-PE1-Pad98) -> /MCU/ICOM_AUX1
- U8 pad R7: /FPGA/FPGA_USART1_TX -> unconnected-(U8F-PB6A-PadR7)
- U8 pad T6: /FPGA/FPGA_USART1_RX -> unconnected-(U8F-PB4A-PadT6)
Other:
- board size 186.6 x 196 mm -> 208.3 x 196 mm
