File: SIGMAGE_HW/SIGMAGE/SIGMAGE.kicad_pcb (KiCad board)
At the start: 2 copper layers, 208.3 x 196 mm, 749 parts, among them J1 UJ31CHG2SMTTR, J10 SJ63073E, J11 SJ63073E, J12 DF40C-40DS-0.4V_51, J13 DF40C-40DP-0.4V_51, J14 DF40C-40DS-0.4V_51, J18 HTSW10107GD, J19 HTSW10107GD, J2 SJ63073E, J20 SJ63073E, J21 SJ63073E, J22 HTSW10107GD, J23 HTSW10107GD, J24 SJ63073E, J25 SJ63073E, J26 HTSW10107GD, J27 HTSW10107GD, J3 TSW10607GS, J4 SJ63073E, J5 TSW10607GS, J6 TSW10607GS, J7 473521001, J8 DF40C-40DP-0.4V_51, J9 TSW10607GS, U1 MAX8902BATA/V+T, U10 PCM5102APWR, U11 TPS62130RGTT, U12 TPS62130RGTT, U13 ESDR0502NMUTBG, U14 93LC56-I/SN, U15 STM32F407VGTx, U16 OPA1612AIDRGR, U17 OPA1612AIDRGR, U18 PCM1803ADB, U19 PCM1803ADB, U2 MAX8902BATA/V+T, U20 PCM5102APWR, U21 PCM5102APWR, U22 EC11E183440C, U23 EC11E183440C, U24 EC11E183440C, U25 EC11E183440C, U26 EC11E183440C, U27 EC11E183440C, U28 EC11E183440C, U29 EC11E183440C, U3 PCM5102APWR, U30 EC11E183440C, U31 MAX8902BATA/V+T, U32 EC11E183440C, U33 EC11E183440C, U34 EC11E183440C, U35 EC11E183440C, U36 EC11E183440C, U37 EC11E183440C, U38 EC11E183440C, U39 EC11E183440C, U4 OPA1612AIDRGR, U40 EC11E183440C, U41 MMBT2222A, U42 TPS62130RGTT, U5 PCM1803ADB, U6 OPA1612AIDRGR, U7 PCM1803ADB, U8 LFE5U25F6BG256I, U9 FT2232HLTRAY, X1 STDCSU18M

Commit message: basic layout
Parts:
- C88: footprint Capacitor_SMD:C_1206_3216Metric -> Capacitor_SMD:C_0603_1608Metric
- J10, J11, J18, J19, J2, J20, J21, J22, J23, J24, J25, J26, J27, J3, J4, J5, J6, J9: moved to B.Cu
- J12, J14: value DF40C-40DS-0.4V_51 -> 61306421821; footprint SIGMAGE:DF40C40DS04V51 -> SIGMAGE:61306421821; moved to B.Cu
- J13, J8: value DF40C-40DP-0.4V_51 -> 61306421121; footprint SIGMAGE:DF40C40DP04V51 -> SIGMAGE:61306421121
- moved R138 342.0 mm to (-195.0, 105.6)
- moved R139 342.0 mm to (-195.0, 108.1)
- moved R140 342.0 mm to (-195.0, 110.6)
- moved R141 342.0 mm to (-195.0, 113.1)
- moved R142 342.0 mm to (-195.0, 115.6)
- moved R143 342.0 mm to (-195.0, 118.1)
- moved R144 342.0 mm to (-195.0, 120.6)
- moved R145 342.0 mm to (-195.0, 123.1)
- moved R146 342.0 mm to (-195.0, 125.6)
- moved R117 342.0 mm to (-207.0, 120.6)
- moved R118 342.0 mm to (-207.0, 123.1)
- moved R119 342.0 mm to (-207.0, 125.6)
- moved R120 342.0 mm to (-203.0, 105.6)
- moved R121 342.0 mm to (-203.0, 108.1)
- moved R122 342.0 mm to (-203.0, 110.6)
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Connections:
- net /ADC/ADC1_BCK renamed 0_ADC1_BCK
- net /ADC/ADC1_BYPAS renamed 0_ADC1_PYPAS
- net /ADC/ADC1_DOUT renamed 0_ADC1_DOUT
- net /ADC/ADC1_FMT0 renamed 0_ADC1_FMT0
- net /ADC/ADC1_FMT1 renamed 0_ADC1_FMT1
- net /ADC/ADC1_LRCK renamed 0_ADC1_LRCK
- net /ADC/ADC1_MODE0 renamed 0_ADC1_MODE0
- net /ADC/ADC1_MODE1 renamed 0_ADC1_MODE1
- net /ADC/ADC1_OSR renamed 0_ADC1_OSR
- net /ADC/ADC1_PDWN renamed 0_ADC1_PDWN
- net /ADC/ADC1_SCKI renamed 0_ADC1_SCKI
- net /ADC/ADC2_BCK renamed 0_ADC2_BCK
- net /ADC/ADC2_BYPAS renamed 0_ADC2_PYPAS
- net /ADC/ADC2_DOUT renamed 0_ADC2_DOUT
- net /ADC/ADC2_FMT0 renamed 0_ADC2_FMT0
- net /ADC/ADC2_FMT1 renamed 0_ADC2_FMT1
- net /ADC/ADC2_LRCK renamed 0_ADC2_LRCK
- net /ADC/ADC2_MODE0 renamed 0_ADC2_MODE0
- net /ADC/ADC2_MODE1 renamed 0_ADC2_MODE1
- net /ADC/ADC2_OSR renamed 0_ADC2_OSR
- net /ADC/ADC2_PDWN renamed 0_ADC2_PDWN
- net /ADC/ADC2_SCKI renamed 0_ADC2_SCKI
- net /ADC/ADC3_BCK renamed 0_ADC3_BCK
- net /ADC/ADC3_BYPAS renamed 0_ADC3_PYPAS
- net /ADC/ADC3_DOUT renamed 0_ADC3_DOUT
- net /ADC/ADC3_FMT0 renamed 0_ADC3_FMT0
- net /ADC/ADC3_FMT1 renamed 0_ADC3_FMT1
- net /ADC/ADC3_LRCK renamed 0_ADC3_LRCK
- net /ADC/ADC3_MODE0 renamed 0_ADC3_MODE0
- net /ADC/ADC3_MODE1 renamed 0_ADC3_MODE1
- net /ADC/ADC3_OSR renamed 0_ADC3_OSR
- net /ADC/ADC3_PDWN renamed 0_ADC3_PDWN
- net /ADC/ADC3_SCKI renamed 0_ADC3_SCKI
- net /ADC/ADC4_BCK renamed 0_ADC4_BCK
- net /ADC/ADC4_BYPAS renamed 0_ADC4_PYPAS
- net /ADC/ADC4_DOUT renamed 0_ADC4_DOUT
- net /ADC/ADC4_FMT0 renamed 0_ADC4_FMT0
- net /ADC/ADC4_FMT1 renamed 0_ADC4_FMT1
- net /ADC/ADC4_LRCK renamed 0_ADC4_LRCK
- net /ADC/ADC4_MODE0 renamed 0_ADC4_MODE0
- net /ADC/ADC4_MODE1 renamed 0_ADC4_MODE1
- net /ADC/ADC4_OSR renamed 0_ADC4_OSR
- net /ADC/ADC4_PDWN renamed 0_ADC4_PDWN
- net /ADC/ADC4_SCKI renamed 0_ADC4_SCKI
- net /ADC/AN_IN1_L renamed 0_AN_IN1_L
- net /ADC/AN_IN1_R renamed 0_AN_IN1_R
- net /ADC/AN_IN2_L renamed 0_AN_IN2_L
- net /ADC/AN_IN2_R renamed 0_AN_IN2_R
- net /ADC/AN_IN3_L renamed 0_AN_IN3_L
- net /ADC/AN_IN3_R renamed 0_AN_IN3_R
- net /ADC/AN_IN4_L renamed 0_AN_IN4_L
- net /ADC/AN_IN4_R renamed 0_AN_IN4_R
- net /BTN/SW1 renamed 1_SW1
- net /BTN/SW10 renamed 1_SW10
- net /BTN/SW11 renamed 1_SW11
- net /BTN/SW12 renamed 1_SW12
- net /BTN/SW2 renamed 1_SW2
- net /BTN/SW3 renamed 1_SW3
- net /BTN/SW4 renamed 1_SW4
- net /BTN/SW5 renamed 1_SW5
- net /BTN/SW6 renamed 1_SW6
- net /BTN/SW7 renamed 1_SW7
- net /BTN/SW8 renamed 1_SW8
- net /BTN/SW9 renamed 1_SW9
- net /DAC/DAC1_CK renamed 0_DAC1_CK
- net /DAC/DAC1_DEMP renamed 0_DAC1_DEMP
- net /DAC/DAC1_FLT renamed 0_DAC1_FLT
- net /DAC/DAC1_FMT renamed 0_DAC1_FMT
- net /DAC/DAC1_SCK renamed 0_DAC1_SCK
- net /DAC/DAC1_SD renamed 0_DAC1_SD
- net /DAC/DAC1_WS renamed 0_DAC1_WS
- net /DAC/DAC1_XSMT renamed 0_DAC1_XSMT
- net /DAC/DAC2_CK renamed 0_DAC2_CK
- net /DAC/DAC2_DEMP renamed 0_DAC2_DEMP
- net /DAC/DAC2_FLT renamed 0_DAC2_FLT
- net /DAC/DAC2_FMT renamed 0_DAC2_FMT
- net /DAC/DAC2_SCK renamed 0_DAC2_SCK
- net /DAC/DAC2_SD renamed 0_DAC2_SD
- net /DAC/DAC2_WS renamed 0_DAC2_WS
- net /DAC/DAC2_XSMT renamed 0_DAC2_XSMT
- net /DAC/DAC3_CK renamed 0_DAC3_CK
- net /DAC/DAC3_DEMP renamed 0_DAC3_DEMP
- net /DAC/DAC3_FLT renamed 0_DAC3_FLT
- net /DAC/DAC3_FMT renamed 0_DAC3_FMT
- net /DAC/DAC3_SCK renamed 0_DAC3_SCK
- net /DAC/DAC3_SD renamed 0_DAC3_SD
- net /DAC/DAC3_WS renamed 0_DAC3_WS
- net /DAC/DAC3_XSMT renamed 0_DAC3_XSMT
- net /DAC/DAC4_CK renamed 0_DAC4_CK
- net /DAC/DAC4_DEMP renamed 0_DAC4_DEMP
- net /DAC/DAC4_FLT renamed 0_DAC4_FLT
- net /DAC/DAC4_FMT renamed 0_DAC4_FMT
- net /DAC/DAC4_SCK renamed 0_DAC4_SCK
- net /DAC/DAC4_SD renamed 0_DAC4_SD
- net /DAC/DAC4_WS renamed 0_DAC4_WS
- net /DAC/DAC4_XSMT renamed 0_DAC4_XSMT
- net /ENC/RE10_A renamed 1_RE10_A
- net /ENC/RE10_B renamed 1_RE10_B
- net /ENC/RE10_C renamed 1_RE10_C
- net /ENC/RE11_A renamed 1_RE11_A
- net /ENC/RE11_B renamed 1_RE11_B
- net /ENC/RE11_C renamed 1_RE11_C
- net /ENC/RE12_A renamed 1_RE12_A
- net /ENC/RE12_B renamed 1_RE12_B
- net /ENC/RE12_C renamed 1_RE12_C
- net /ENC/RE13_A renamed 1_RE13_A
- net /ENC/RE13_B renamed 1_RE13_B
- net /ENC/RE13_C renamed 1_RE13_C
- net /ENC/RE14_A renamed 1_RE14_A
- net /ENC/RE14_B renamed 1_RE14_B
- net /ENC/RE14_C renamed 1_RE14_C
- net /ENC/RE15_A renamed 1_RE15_A
- net /ENC/RE15_B renamed 1_RE15_B
- net /ENC/RE15_C renamed 1_RE15_C
- net /ENC/RE16_A renamed 1_RE16_A
- net /ENC/RE16_B renamed 1_RE16_B
- net /ENC/RE16_C renamed 1_RE16_C
- net /ENC/RE17_A renamed 1_RE17_A
- net /ENC/RE17_B renamed 1_RE17_B
- net /ENC/RE17_C renamed 1_RE17_C
- net /ENC/RE18_A renamed 1_RE18_A
- net /ENC/RE18_B renamed 1_RE18_B
- net /ENC/RE18_C renamed 1_RE18_C
- net /ENC/RE1_A renamed 1_RE1_A
- net /ENC/RE1_B renamed 1_RE1_B
- net /ENC/RE1_C renamed 1_RE1_C
- net /ENC/RE2_A renamed 1_RE2_A
- net /ENC/RE2_B renamed 1_RE2_B
- net /ENC/RE2_C renamed 1_RE2_C
- net /ENC/RE3_A renamed 1_RE3_A
- net /ENC/RE3_B renamed 1_RE3_B
- net /ENC/RE3_C renamed 1_RE3_C
- net /ENC/RE4_A renamed 1_RE4_A
- net /ENC/RE4_B renamed 1_RE4_B
- net /ENC/RE4_C renamed 1_RE4_C
- net /ENC/RE5_A renamed 1_RE5_A
- net /ENC/RE5_B renamed 1_RE5_B
- net /ENC/RE5_C renamed 1_RE5_C
- net /ENC/RE6_A renamed 1_RE6_A
- net /ENC/RE6_B renamed 1_RE6_B
- net /ENC/RE6_C renamed 1_RE6_C
- net /ENC/RE7_A renamed 1_RE7_A
- net /ENC/RE7_B renamed 1_RE7_B
- net /ENC/RE7_C renamed 1_RE7_C
- net /ENC/RE8_A renamed 1_RE8_A
- net /ENC/RE8_B renamed 1_RE8_B
- net /ENC/RE8_C renamed 1_RE8_C
- net /ENC/RE9_A renamed 1_RE9_A
- net /ENC/RE9_B renamed 1_RE9_B
- net /ENC/RE9_C renamed 1_RE9_C
- net /FPGA/FPGA_CFG0 renamed 0_FPGA_CFG0
- net /FPGA/FPGA_CFG1 renamed 0_FPGA_CFG1
- net /FPGA/FPGA_CFG2 renamed 0_FPGA_CFG2
- net /FPGA/FPGA_DONE renamed 0_FPGA_DONE
- net /FPGA/FPGA_HOLDN renamed 0_FPGA_HOLDN
- net /FPGA/FPGA_INITN renamed 0_FPGA_INITN
- net /FPGA/FPGA_PROGRAMN renamed 0_FPGA_PROGRAMN
- net /FPGA/FPGA_USART1_RX renamed 0_FPGA_USART1_RX
- net /FPGA/FPGA_USART1_TX renamed 0_FPGA_USART1_TX
- net /LED/T_LED_C1 renamed 1_LED_C1
- net /LED/T_LED_C10 renamed 1_LED_C10
- net /LED/T_LED_C11 renamed 1_LED_C11
- net /LED/T_LED_C12 renamed 1_LED_C12
- net /LED/T_LED_C13 renamed 1_LED_C13
- net /LED/T_LED_C14 renamed 1_LED_C14
- net /LED/T_LED_C15 renamed 1_LED_C15
- net /LED/T_LED_C16 renamed 1_LED_C16
- net /LED/T_LED_C2 renamed 1_LED_C2
- net /LED/T_LED_C3 renamed 1_LED_C3
- net /LED/T_LED_C4 renamed 1_LED_C4
- net /LED/T_LED_C5 renamed 1_LED_C5
- net /LED/T_LED_C6 renamed 1_LED_C6
- net /LED/T_LED_C7 renamed 1_LED_C7
- net /LED/T_LED_C8 renamed 1_LED_C8
- net /LED/T_LED_C9 renamed 1_LED_C9
- net /LED/T_LED_R1 renamed 1_LED_R1
- net /LED/T_LED_R10 renamed 1_LED_R10
- net /LED/T_LED_R11 renamed 1_LED_R11
- net /LED/T_LED_R12 renamed 1_LED_R12
- net /LED/T_LED_R13 renamed 1_LED_R13
- net /LED/T_LED_R14 renamed 1_LED_R14
- net /LED/T_LED_R15 renamed 1_LED_R15
- net /LED/T_LED_R16 renamed 1_LED_R16
- net /LED/T_LED_R2 renamed 1_LED_R2
- net /LED/T_LED_R3 renamed 1_LED_R3
- net /LED/T_LED_R4 renamed 1_LED_R4
- net /LED/T_LED_R5 renamed 1_LED_R5
- net /LED/T_LED_R6 renamed 1_LED_R6
- net /LED/T_LED_R7 renamed 1_LED_R7
- net /LED/T_LED_R8 renamed 1_LED_R8
- net /LED/T_LED_R9 renamed 1_LED_R9
- net /MCU/ICOM_AUX0 renamed 0_ICOM_AUX0
- net /MCU/ICOM_AUX1 renamed 0_ICOM_AUX1
- net /MCU/ICOM_AUX10 renamed 0_ICOM_AUX10
- net /MCU/ICOM_AUX11 renamed 0_ICOM_AUX11
- net /MCU/ICOM_AUX12 renamed 0_ICOM_AUX12
- net /MCU/ICOM_AUX13 renamed 0_ICOM_AUX13
- net /MCU/ICOM_AUX14 renamed 0_ICOM_AUX14
- net /MCU/ICOM_AUX15 renamed 0_ICOM_AUX15
- net /MCU/ICOM_AUX2 renamed 0_ICOM_AUX2
- net /MCU/ICOM_AUX3 renamed 0_ICOM_AUX3
- net /MCU/ICOM_AUX4 renamed 0_ICOM_AUX4
- net /MCU/ICOM_AUX5 renamed 0_ICOM_AUX5
- net /MCU/ICOM_AUX6 renamed 0_ICOM_AUX6
- net /MCU/ICOM_AUX7 renamed 0_ICOM_AUX7
- net /MCU/ICOM_AUX8 renamed 0_ICOM_AUX8
- net /MCU/ICOM_AUX9 renamed 0_ICOM_AUX9
- net /MCU/ICOM_USART3_RX renamed 0_ICOM_USART3_RX
- net /MCU/ICOM_USART3_TX renamed 0_ICOM_USART3_TX
- net /MCU/MCU_USART1_RX renamed 0_MCU_USART1_RX
- net /MCU/MCU_USART1_TX renamed 0_MCU_USART1_TX
- J1 pad A6: /USB/USB_DP -> 0_USB_DP
- J1 pad A7: /USB/USB_DN -> 0_USB_DN
- J1 pad B6: /USB/USB_DP -> 0_USB_DP
- J1 pad B7: /USB/USB_DN -> 0_USB_DN
- J12 pad 1: /MEZZ/B_LED_C1 -> unconnected-(J12-Pad1)
- J12 pad 10: /MEZZ/B_LED_R5 -> unconnected-(J12-Pad10)
- J12 pad 11: /MEZZ/B_LED_C6 -> unconnected-(J12-Pad11)
- J12 pad 12: /MEZZ/B_LED_R6 -> unconnected-(J12-Pad12)
- J12 pad 13: /MEZZ/B_LED_C7 -> unconnected-(J12-Pad13)
- J12 pad 14: /MEZZ/B_LED_R7 -> unconnected-(J12-Pad14)
- J12 pad 15: /MEZZ/B_LED_C8 -> unconnected-(J12-Pad15)
- J12 pad 16: /MEZZ/B_LED_R8 -> unconnected-(J12-Pad16)
- J12 pad 17: /MEZZ/B_LED_C9 -> unconnected-(J12-Pad17)
- J12 pad 18: /MEZZ/B_LED_R9 -> unconnected-(J12-Pad18)
- J12 pad 19: /MEZZ/B_LED_C10 -> unconnected-(J12-Pad19)
- J12 pad 2: /MEZZ/B_LED_R1 -> unconnected-(J12-Pad2)
- J12 pad 20: /MEZZ/B_LED_R10 -> unconnected-(J12-Pad20)
- J12 pad 21: /MEZZ/B_LED_C11 -> unconnected-(J12-Pad21)
- J12 pad 22: /MEZZ/B_LED_R11 -> unconnected-(J12-Pad22)
- J12 pad 23: /MEZZ/B_LED_C12 -> unconnected-(J12-Pad23)
- J12 pad 24: /MEZZ/B_LED_R12 -> unconnected-(J12-Pad24)
- J12 pad 25: /MEZZ/B_LED_C13 -> unconnected-(J12-Pad25)
- J12 pad 26: /MEZZ/B_LED_R13 -> unconnected-(J12-Pad26)
- J12 pad 27: /MEZZ/B_LED_C14 -> unconnected-(J12-Pad27)
- J12 pad 28: /MEZZ/B_LED_R14 -> unconnected-(J12-Pad28)
- J12 pad 29: /MEZZ/B_LED_C15 -> unconnected-(J12-Pad29)
- J12 pad 3: /MEZZ/B_LED_C2 -> unconnected-(J12-Pad3)
- J12 pad 30: /MEZZ/B_LED_R15 -> unconnected-(J12-Pad30)
- J12 pad 31: /MEZZ/B_LED_C16 -> unconnected-(J12-Pad31)
- J12 pad 32: /MEZZ/B_LED_R16 -> unconnected-(J12-Pad32)
- J12 pad 4: /MEZZ/B_LED_R2 -> unconnected-(J12-Pad4)
- J12 pad 5: /MEZZ/B_LED_C3 -> unconnected-(J12-Pad5)
- J12 pad 6: /MEZZ/B_LED_R3 -> unconnected-(J12-Pad6)
- J12 pad 7: /MEZZ/B_LED_C4 -> unconnected-(J12-Pad7)
- J12 pad 8: /MEZZ/B_LED_R4 -> unconnected-(J12-Pad8)
- J12 pad 9: /MEZZ/B_LED_C5 -> unconnected-(J12-Pad9)
- J3 pad 2: /USB/FPGA_JTAG_TMS -> 0_FPGA_JTAG_TMS
- J3 pad 3: /USB/FPGA_JTAG_TDO -> 0_FPGA_JTAG_TDO
- J3 pad 4: /USB/FPGA_JTAG_TDI -> 0_FPGA_JTAG_TDI
- J3 pad 5: /USB/FPGA_JTAG_TCK -> 0_FPGA_JTAG_TCK
- J6 pad 2: /USB/MCU_JTAG_TMS -> 0_MCU_JTAG_TMS
- J6 pad 3: /USB/MCU_JTAG_TDO -> 0_MCU_JTAG_TDO
- J6 pad 4: /USB/MCU_JTAG_TDI -> 0_MCU_JTAG_TDI
- J6 pad 5: /USB/MCU_JTAG_TCK -> 0_MCU_JTAG_TCK
- J7 pad 2: /SDCARD/SDCARD_SPI_CS -> 0_SDCARD_SPI_CS
- J7 pad 3: /SDCARD/SDCARD_SPI_MOSI -> 0_SDCARD_SPI_MOSI
- J7 pad 5: /SDCARD/SDCARD_SPI_SCK -> 0_SDCARD_SPI_SCK
- J7 pad 7: /SDCARD/SDCARD_SPI_MISO -> 0_SDCARD_SPI_MISO
- J8 pad 1: /MEZZ/T_LED_C1 -> unconnected-(J8-Pad1)
- J8 pad 10: /MEZZ/T_LED_R5 -> unconnected-(J8-Pad10)
- J8 pad 11: /MEZZ/T_LED_C6 -> unconnected-(J8-Pad11)
- J8 pad 12: /MEZZ/T_LED_R6 -> unconnected-(J8-Pad12)
- J8 pad 13: /MEZZ/T_LED_C7 -> unconnected-(J8-Pad13)
- J8 pad 14: /MEZZ/T_LED_R7 -> unconnected-(J8-Pad14)
- J8 pad 15: /MEZZ/T_LED_C8 -> unconnected-(J8-Pad15)
- J8 pad 16: /MEZZ/T_LED_R8 -> unconnected-(J8-Pad16)
- J8 pad 17: /MEZZ/T_LED_C9 -> unconnected-(J8-Pad17)
- J8 pad 18: /MEZZ/T_LED_R9 -> unconnected-(J8-Pad18)
- J8 pad 19: /MEZZ/T_LED_C10 -> unconnected-(J8-Pad19)
- J8 pad 2: /MEZZ/T_LED_R1 -> unconnected-(J8-Pad2)
- J8 pad 20: /MEZZ/T_LED_R10 -> unconnected-(J8-Pad20)
- J8 pad 21: /MEZZ/T_LED_C11 -> unconnected-(J8-Pad21)
- J8 pad 22: /MEZZ/T_LED_R11 -> unconnected-(J8-Pad22)
- J8 pad 23: /MEZZ/T_LED_C12 -> unconnected-(J8-Pad23)
- J8 pad 24: /MEZZ/T_LED_R12 -> unconnected-(J8-Pad24)
- J8 pad 25: /MEZZ/T_LED_C13 -> unconnected-(J8-Pad25)
- J8 pad 26: /MEZZ/T_LED_R13 -> unconnected-(J8-Pad26)
- J8 pad 27: /MEZZ/T_LED_C14 -> unconnected-(J8-Pad27)
- J8 pad 28: /MEZZ/T_LED_R14 -> unconnected-(J8-Pad28)
- J8 pad 29: /MEZZ/T_LED_C15 -> unconnected-(J8-Pad29)
- J8 pad 3: /MEZZ/T_LED_C2 -> unconnected-(J8-Pad3)
- J8 pad 30: /MEZZ/T_LED_R15 -> unconnected-(J8-Pad30)
- J8 pad 31: /MEZZ/T_LED_C16 -> unconnected-(J8-Pad31)
- J8 pad 32: /MEZZ/T_LED_R16 -> unconnected-(J8-Pad32)
- J8 pad 4: /MEZZ/T_LED_R2 -> unconnected-(J8-Pad4)
- J8 pad 5: /MEZZ/T_LED_C3 -> unconnected-(J8-Pad5)
- J8 pad 6: /MEZZ/T_LED_R3 -> unconnected-(J8-Pad6)
- J8 pad 7: /MEZZ/T_LED_C4 -> unconnected-(J8-Pad7)
- J8 pad 8: /MEZZ/T_LED_R4 -> unconnected-(J8-Pad8)
- J8 pad 9: /MEZZ/T_LED_C5 -> unconnected-(J8-Pad9)
- R107 pad 1: /SDCARD/SDCARD_SPI_CS -> 0_SDCARD_SPI_CS
- R108 pad 1: /SDCARD/SDCARD_SPI_MOSI -> 0_SDCARD_SPI_MOSI
- R109 pad 1: /SDCARD/SDCARD_SPI_MISO -> 0_SDCARD_SPI_MISO
- R113 pad 1: /FPGA/FPGA_SPI_CLK -> 0_FPGA_SPI_CLK
- R114 pad 1: /FPGA/FPGA_SPI_MISO -> 0_FPGA_SPI_MISO
- R115 pad 1: /FPGA/FPGA_SPI_MOSI -> 0_FPGA_SPI_MOSI
- R116 pad 1: /FPGA/FPGA_SPI_CS -> 0_FPGA_SPI_CS
- R185 pad 1: /SDCARD/SDCARD_SPI_SCK -> 0_SDCARD_SPI_SCK
- R28 pad 2: /USB/FPGA_JTAG_TCK -> 0_FPGA_JTAG_TCK
- R29 pad 1: /USB/FPGA_JTAG_TDI -> 0_FPGA_JTAG_TDI
- R30 pad 1: /USB/FPGA_JTAG_TDO -> 0_FPGA_JTAG_TDO
- R31 pad 1: /USB/FPGA_JTAG_TMS -> 0_FPGA_JTAG_TMS
- R59 pad 1: /USB/MCU_JTAG_TDI -> 0_MCU_JTAG_TDI
- R60 pad 2: /USB/MCU_JTAG_TCK -> 0_MCU_JTAG_TCK
- R61 pad 1: /USB/MCU_JTAG_TDO -> 0_MCU_JTAG_TDO
- R62 pad 1: /USB/MCU_JTAG_TMS -> 0_MCU_JTAG_TMS
- U13 pad 2: /USB/USB_DP -> 0_USB_DP
- U13 pad 3: /USB/USB_DN -> 0_USB_DN
- U13 pad 4: /USB/USB_DN -> 0_USB_DN
- U13 pad 5: /USB/USB_DP -> 0_USB_DP
- U15 pad 29: /MCU/SDCARD_SPI_CS -> 0_SDCARD_SPI_CS
- U15 pad 30: /MCU/SDCARD_SPI_SCK -> 0_SDCARD_SPI_SCK
- U15 pad 31: /MCU/SDCARD_SPI_MISO -> 0_SDCARD_SPI_MISO
- U15 pad 32: /MCU/SDCARD_SPI_MOSI -> 0_SDCARD_SPI_MOSI
- U15 pad 51: /MCU/FPGA_SPI_CS -> 0_FPGA_SPI_CS
- U15 pad 52: /MCU/FPGA_SPI_CLK -> 0_FPGA_SPI_CLK
- U15 pad 53: /MCU/FPGA_SPI_MISO -> 0_FPGA_SPI_MISO
- U15 pad 54: /MCU/FPGA_SPI_MOSI -> 0_FPGA_SPI_MOSI
- U15 pad 72: /MCU/MCU_JTAG_TMS -> 0_MCU_JTAG_TMS
- U15 pad 76: /MCU/MCU_JTAG_TCK -> 0_MCU_JTAG_TCK
- U15 pad 77: /MCU/MCU_JTAG_TDI -> 0_MCU_JTAG_TDI
- U15 pad 89: /MCU/MCU_JTAG_TDO -> 0_MCU_JTAG_TDO
- U8 pad M10: /FPGA/FPGA_JTAG_TDO -> 0_FPGA_JTAG_TDO
- U8 pad N9: /FPGA/FPGA_SPI_CLK -> 0_FPGA_SPI_CLK
- U8 pad R11: /FPGA/FPGA_JTAG_TDI -> 0_FPGA_JTAG_TDI
- U8 pad R8: /FPGA/FPGA_SPI_CS -> 0_FPGA_SPI_CS
- U8 pad T10: /FPGA/FPGA_JTAG_TCK -> 0_FPGA_JTAG_TCK
- U8 pad T11: /FPGA/FPGA_JTAG_TMS -> 0_FPGA_JTAG_TMS
- U8 pad T7: /FPGA/FPGA_SPI_MISO -> 0_FPGA_SPI_MISO
- U8 pad T8: /FPGA/FPGA_SPI_MOSI -> 0_FPGA_SPI_MOSI
- U9 pad 16: /USB/FPGA_JTAG_TCK -> 0_FPGA_JTAG_TCK
- U9 pad 17: /USB/FPGA_JTAG_TDI -> 0_FPGA_JTAG_TDI
- U9 pad 18: /USB/FPGA_JTAG_TDO -> 0_FPGA_JTAG_TDO
- U9 pad 19: /USB/FPGA_JTAG_TMS -> 0_FPGA_JTAG_TMS
- U9 pad 38: /USB/MCU_JTAG_TCK -> 0_MCU_JTAG_TCK
- U9 pad 39: /USB/MCU_JTAG_TDI -> 0_MCU_JTAG_TDI
- U9 pad 40: /USB/MCU_JTAG_TDO -> 0_MCU_JTAG_TDO
- U9 pad 41: /USB/MCU_JTAG_TMS -> 0_MCU_JTAG_TMS
Routing:
- net (no net): vias 0 -> 8
Other:
- board size 208.3 x 196 mm -> 270 x 170 mm

Commit message: uga uga
Parts:
- removed C193, C194, C195, C196, C197, C198, C199: 100n, Capacitor_SMD:C_0603_1608Metric
- removed R138, R139, R140, R141, R142, R143, R144, R145, R146, R162, R163, R164, R165, R166, R167, R168: 10k, Resistor_SMD:R_0603_1608Metric
- removed S10, S11, S12, S6, S7, S8, S9: TL2201EEYA, SIGMAGE:TL2201EEYA
- removed U38, U39, U40: EC11E183440C, SIGMAGE:EC11E183440C
- C12, C125, C126, C127, C128, C129, C13, C130, C131, C132, C133, C134, C135, C136, C137, C138, C139, C140, C141, C142, C165, C166, C167, C168, C173, C174, C175, C176, C179, C18, C180, C181, C182, C183, C184, C185, C186, C19, C20, C21, C22, C23, C62, C63, C82, C83, C89, C90: footprint Capacitor_SMD:C_1206_3216Metric -> Resistor_SMD:R_0603_1608Metric
- moved U37 464.8 mm to (281.5, 201.2)
- moved U36 459.7 mm to (257.5, 201.2)
- moved U35 454.9 mm to (233.8, 201.2)
- moved D261 410.8 mm to (311.2, 74.8)
- moved D262 410.4 mm to (311.2, 78.2)
- moved U41 409.9 mm to (311.2, 68.2), turned to 180 degrees
- moved D278 341.0 mm to (300.8, 77.8), turned to -90 degrees
- moved D277 336.8 mm to (296.8, 77.8), turned to -90 degrees
- moved R184 336.5 mm to (300.8, 74.8), turned to -90 degrees
- moved D276 332.7 mm to (292.8, 77.8), turned to -90 degrees
- moved R183 332.4 mm to (296.8, 74.8), turned to -90 degrees
- moved D274 329.6 mm to (284.8, 77.8), turned to -90 degrees
- moved D275 328.5 mm to (288.8, 77.8), turned to -90 degrees
- moved R182 328.3 mm to (292.8, 74.8), turned to -90 degrees
- moved D273 325.3 mm to (280.8, 77.8), turned to -90 degrees
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Connections:
- D263 pad 2: Net-(D263-A) -> 1_LED0
- D264 pad 2: Net-(D264-A) -> 1_LED1
- D265 pad 2: Net-(D265-A) -> 1_LED2
- D266 pad 2: Net-(D266-A) -> 1_LED3
- D267 pad 2: Net-(D267-A) -> 1_LED4
- D268 pad 2: Net-(D268-A) -> 1_LED5
- D269 pad 2: Net-(D269-A) -> 1_LED6
- D270 pad 2: Net-(D270-A) -> 1_LED7
- D271 pad 2: Net-(D271-A) -> 1_LED8
- D272 pad 2: Net-(D272-A) -> 1_LED9
- D273 pad 2: Net-(D273-A) -> 1_LED10
- D274 pad 2: Net-(D274-A) -> 1_LED11
- D275 pad 2: Net-(D275-A) -> 1_LED12
- D276 pad 2: Net-(D276-A) -> 1_LED13
- D277 pad 2: Net-(D277-A) -> 1_LED14
- D278 pad 2: Net-(D278-A) -> 1_LED15
- J12 pad 1: unconnected-(J12-Pad1) -> 1_RE5_B
- J12 pad 10: unconnected-(J12-Pad10) -> 1_LED11
- J12 pad 11: unconnected-(J12-Pad11) -> 1_RE12_C
- J12 pad 12: unconnected-(J12-Pad12) -> 1_LED10
- J12 pad 13: unconnected-(J12-Pad13) -> 1_RE11_B
- J12 pad 14: unconnected-(J12-Pad14) -> 1_LED9
- J12 pad 15: unconnected-(J12-Pad15) -> 1_RE11_A
- J12 pad 16: unconnected-(J12-Pad16) -> 1_LED8
- J12 pad 17: unconnected-(J12-Pad17) -> 1_RE11_C
- J12 pad 18: unconnected-(J12-Pad18) -> 1_LED7
- J12 pad 2: unconnected-(J12-Pad2) -> 1_LED15
- J12 pad 20: unconnected-(J12-Pad20) -> 1_LED6
- J12 pad 3: unconnected-(J12-Pad3) -> 1_RE5_A
- J12 pad 36: unconnected-(J12-Pad36) -> 1_LED5
- J12 pad 37: unconnected-(J12-Pad37) -> 1_SW5
- J12 pad 38: unconnected-(J12-Pad38) -> 1_LED4
- J12 pad 39: unconnected-(J12-Pad39) -> 1_SW4
- J12 pad 4: unconnected-(J12-Pad4) -> 1_LED14
- J12 pad 40: unconnected-(J12-Pad40) -> 1_LED3
- J12 pad 41: unconnected-(J12-Pad41) -> 1_SW3
- J12 pad 42: unconnected-(J12-Pad42) -> 1_LED2
- J12 pad 43: unconnected-(J12-Pad43) -> 1_SW2
- J12 pad 44: unconnected-(J12-Pad44) -> 1_LED1
- J12 pad 45: unconnected-(J12-Pad45) -> 1_SW1
- J12 pad 46: unconnected-(J12-Pad46) -> 1_LED0
- J12 pad 47: unconnected-(J12-Pad47) -> 1_RE10_B
- J12 pad 48: unconnected-(J12-Pad48) -> 1_RE10_A
- J12 pad 49: unconnected-(J12-Pad49) -> 1_RE10_C
- J12 pad 5: unconnected-(J12-Pad5) -> 1_RE5_C
- J12 pad 50: unconnected-(J12-Pad50) -> 1_RE4_B
- J12 pad 51: unconnected-(J12-Pad51) -> 1_RE4_A
- J12 pad 52: unconnected-(J12-Pad52) -> 1_RE4_C
- J12 pad 53: unconnected-(J12-Pad53) -> 1_RE3_B
- J12 pad 54: unconnected-(J12-Pad54) -> 1_RE3_A
- J12 pad 55: unconnected-(J12-Pad55) -> 1_RE3_C
- J12 pad 56: unconnected-(J12-Pad56) -> 1_RE2_B
- J12 pad 57: unconnected-(J12-Pad57) -> 1_RE2_A
- J12 pad 58: unconnected-(J12-Pad58) -> 1_RE2_C
- J12 pad 59: unconnected-(J12-Pad59) -> 1_RE1_B
- J12 pad 6: unconnected-(J12-Pad6) -> 1_LED13
- J12 pad 60: unconnected-(J12-Pad60) -> 1_RE9_B
- J12 pad 61: unconnected-(J12-Pad61) -> 1_RE1_A
- J12 pad 62: unconnected-(J12-Pad62) -> 1_RE9_C
- J12 pad 63: unconnected-(J12-Pad63) -> 1_RE1_C
- J12 pad 64: unconnected-(J12-Pad64) -> 1_RE9_A
- J12 pad 7: unconnected-(J12-Pad7) -> 1_RE12_B
- J12 pad 8: unconnected-(J12-Pad8) -> 1_LED12
- J12 pad 9: unconnected-(J12-Pad9) -> 1_RE12_A
- J14 pad 15: unconnected-(J14-Pad15) -> 1_RE8_B
- J14 pad 16: unconnected-(J14-Pad16) -> 1_RE8_A
- J14 pad 17: unconnected-(J14-Pad17) -> 1_RE8_C
- J14 pad 18: unconnected-(J14-Pad18) -> 1_RE7_B
- J14 pad 19: unconnected-(J14-Pad19) -> 1_RE7_A
- J14 pad 20: unconnected-(J14-Pad20) -> 1_RE7_C
- J14 pad 21: unconnected-(J14-Pad21) -> 1_RE6_B
- J14 pad 22: unconnected-(J14-Pad22) -> 1_RE6_A
- J14 pad 23: unconnected-(J14-Pad23) -> 1_RE6_C
- J14 pad 24: unconnected-(J14-Pad24) -> 1_RE15_B
- J14 pad 25: unconnected-(J14-Pad25) -> 1_RE15_A
- J14 pad 26: unconnected-(J14-Pad26) -> 1_RE15_C
- J14 pad 27: unconnected-(J14-Pad27) -> 1_RE14_B
- J14 pad 28: unconnected-(J14-Pad28) -> 1_RE14_C
- J14 pad 29: unconnected-(J14-Pad29) -> 1_RE13_C
- J14 pad 30: unconnected-(J14-Pad30) -> 1_RE14_A
- J14 pad 31: unconnected-(J14-Pad31) -> 1_RE13_A
- J14 pad 32: unconnected-(J14-Pad32) -> 1_RE13_B
- J14 pad 33: unconnected-(J14-Pad33) -> 1_LED_C15
- J14 pad 34: unconnected-(J14-Pad34) -> 1_LED_C16
- J14 pad 35: unconnected-(J14-Pad35) -> 1_LED_C13
- J14 pad 36: unconnected-(J14-Pad36) -> 1_LED_C14
- J14 pad 37: unconnected-(J14-Pad37) -> 1_LED_C11
- J14 pad 38: unconnected-(J14-Pad38) -> 1_LED_C12
- J14 pad 39: unconnected-(J14-Pad39) -> 1_LED_C9
- J14 pad 40: unconnected-(J14-Pad40) -> 1_LED_C10
- J14 pad 41: unconnected-(J14-Pad41) -> 1_LED_C7
- J14 pad 42: unconnected-(J14-Pad42) -> 1_LED_C8
- J14 pad 43: unconnected-(J14-Pad43) -> 1_LED_C5
- J14 pad 44: unconnected-(J14-Pad44) -> 1_LED_C6
- J14 pad 45: unconnected-(J14-Pad45) -> 1_LED_C3
- J14 pad 46: unconnected-(J14-Pad46) -> 1_LED_C4
- J14 pad 47: unconnected-(J14-Pad47) -> 1_LED_C1
- J14 pad 48: unconnected-(J14-Pad48) -> 1_LED_C2
- J14 pad 49: unconnected-(J14-Pad49) -> 1_LED_R15
- J14 pad 50: unconnected-(J14-Pad50) -> 1_LED_R16
- J14 pad 51: unconnected-(J14-Pad51) -> 1_LED_R13
- J14 pad 52: unconnected-(J14-Pad52) -> 1_LED_R14
- J14 pad 53: unconnected-(J14-Pad53) -> 1_LED_R11
- J14 pad 54: unconnected-(J14-Pad54) -> 1_LED_R12
- J14 pad 55: unconnected-(J14-Pad55) -> 1_LED_R9
- J14 pad 56: unconnected-(J14-Pad56) -> 1_LED_R10
- J14 pad 57: unconnected-(J14-Pad57) -> 1_LED_R7
- J14 pad 58: unconnected-(J14-Pad58) -> 1_LED_R8
- J14 pad 59: unconnected-(J14-Pad59) -> 1_LED_R5
- J14 pad 60: unconnected-(J14-Pad60) -> 1_LED_R6
- J14 pad 61: unconnected-(J14-Pad61) -> 1_LED_R3
- J14 pad 62: unconnected-(J14-Pad62) -> 1_LED_R4
- J14 pad 63: unconnected-(J14-Pad63) -> 1_LED_R1
- J14 pad 64: unconnected-(J14-Pad64) -> 1_LED_R2
- U15 pad 55: Net-(D271-A) -> 0_LED8
- U15 pad 56: Net-(D272-A) -> 0_LED9
- U15 pad 57: Net-(D273-A) -> 0_LED10
- U15 pad 58: Net-(D274-A) -> 0_LED11
- U15 pad 59: Net-(D275-A) -> 0_LED12
- U15 pad 60: Net-(D276-A) -> 0_LED13
- U15 pad 61: Net-(D277-A) -> 0_LED14
- U15 pad 62: Net-(D278-A) -> 0_LED15
- U15 pad 81: Net-(D263-A) -> 0_LED0
- U15 pad 82: Net-(D264-A) -> 0_LED1
- U15 pad 83: Net-(D265-A) -> 0_LED2
- U15 pad 84: Net-(D266-A) -> 0_LED3
- U15 pad 85: Net-(D267-A) -> 0_LED4
- U15 pad 86: Net-(D268-A) -> 0_LED5
- U15 pad 87: Net-(D269-A) -> 0_LED6
- U15 pad 88: Net-(D270-A) -> 0_LED7
Routing:
- net 1_LED_C16: track 0.00 -> 128.9 mm
- net 1_LED_C15: track 0.00 -> 128.0 mm
- net 1_RE4_B: track 0.00 -> 121.5 mm
- net 1_LED_C14: track 0.00 -> 121.0 mm
- net 1_LED_C13: track 0.00 -> 120.1 mm
- net 1_RE4_A: track 0.00 -> 118.1 mm
- net 1_LED_C12: track 0.00 -> 113.1 mm
- net 1_LED_C11: track 0.00 -> 112.2 mm
- net 1_LED_C1: track 0.00 -> 106.8 mm
- net 1_RE4_C: track 0.00 -> 106.1 mm
- net 1_LED_C10: track 0.00 -> 105.2 mm
- net 1_LED_C9: track 0.00 -> 104.3 mm
- net 1_RE6_C: track 0.00 -> 103.2 mm
- net 1_LED_C2: track 0.00 -> 99.8 mm
- net 1_LED_C3: track 0.00 -> 98.9 mm
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Other:
- copper layers 2 -> 6

Commit message: almost done with tha top part
Parts:
- moved R90 523.1 mm to (309.8, 199.0), turned to -90 degrees
- moved R84 521.2 mm to (309.8, 147.0), turned to -90 degrees
- moved R81 520.8 mm to (309.8, 121.0), turned to -90 degrees
- moved R87 520.5 mm to (309.8, 173.0), turned to -90 degrees
- moved R88 518.9 mm to (304.8, 199.0), turned to -90 degrees
- moved R82 516.4 mm to (304.8, 147.0), turned to -90 degrees
- moved R85 516.2 mm to (304.8, 173.0), turned to -90 degrees
- moved R80 516.0 mm to (304.8, 99.0), turned to 90 degrees
- moved R79 515.8 mm to (304.8, 121.0), turned to -90 degrees
- moved R83 515.8 mm to (304.8, 125.0), turned to 90 degrees
- moved R89 515.4 mm to (304.8, 177.0), turned to 90 degrees
- moved R86 513.6 mm to (304.8, 151.0), turned to 90 degrees
- moved R128 489.6 mm to (286.5, 114.5), turned to -90 degrees
- moved R127 485.5 mm to (281.5, 92.5), turned to 90 degrees
- moved R126 484.5 mm to (281.5, 114.5), turned to -90 degrees
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Connections:
- D262 pad 1: 0_FPGA_INITN -> 1_FPGA_INITN
- J12 pad 1: 1_RE5_B -> 1_FPGA_INITN
- J12 pad 10: 1_LED11 -> 1_LED12
- J12 pad 11: 1_RE12_C -> 1_RE12_A
- J12 pad 12: 1_LED10 -> 1_LED11
- J12 pad 13: 1_RE11_B -> 1_RE12_C
- J12 pad 14: 1_LED9 -> 1_LED10
- J12 pad 15: 1_RE11_A -> 1_RE11_B
- J12 pad 16: 1_LED8 -> 1_LED9
- J12 pad 17: 1_RE11_C -> 1_RE11_A
- J12 pad 18: 1_LED7 -> 1_LED8
- J12 pad 19: unconnected-(J12-Pad19) -> 1_RE11_C
- J12 pad 2: 1_LED15 -> 1_FPGA_DONE
- J12 pad 20: 1_LED6 -> 1_LED7
- J12 pad 21: unconnected-(J12-Pad21) -> DVCC_3V3
- J12 pad 22: unconnected-(J12-Pad22) -> 1_LED6
- J12 pad 23: unconnected-(J12-Pad23) -> DVCC_3V3
- J12 pad 24: unconnected-(J12-Pad24) -> 1_LED5
- J12 pad 25: unconnected-(J12-Pad25) -> DVCC_3V3
- J12 pad 26: unconnected-(J12-Pad26) -> 1_LED4
- J12 pad 27: unconnected-(J12-Pad27) -> DVCC_3V3
- J12 pad 28: unconnected-(J12-Pad28) -> 1_LED3
- J12 pad 29: unconnected-(J12-Pad29) -> DVCC_3V3
- J12 pad 3: 1_RE5_A -> 1_RE5_B
- J12 pad 30: unconnected-(J12-Pad30) -> 1_LED2
- J12 pad 31: unconnected-(J12-Pad31) -> DVCC_3V3
- J12 pad 32: unconnected-(J12-Pad32) -> 1_LED1
- J12 pad 33: unconnected-(J12-Pad33) -> DVCC_3V3
- J12 pad 34: unconnected-(J12-Pad34) -> 1_LED0
- J12 pad 35: unconnected-(J12-Pad35) -> GND
- J12 pad 36: 1_LED5 -> 1_SW5
- J12 pad 37: 1_SW5 -> GND
- J12 pad 38: 1_LED4 -> 1_SW4
- J12 pad 39: 1_SW4 -> GND
- J12 pad 4: 1_LED14 -> 1_LED15
- J12 pad 40: 1_LED3 -> 1_SW3
- J12 pad 41: 1_SW3 -> GND
- J12 pad 42: 1_LED2 -> 1_SW2
- J12 pad 43: 1_SW2 -> GND
- J12 pad 44: 1_LED1 -> 1_SW1
- J12 pad 45: 1_SW1 -> GND
- J12 pad 46: 1_LED0 -> unconnected-(J12-Pad46)
- J12 pad 5: 1_RE5_C -> 1_RE5_A
- J12 pad 6: 1_LED13 -> 1_LED14
- J12 pad 7: 1_RE12_B -> 1_RE5_C
- J12 pad 8: 1_LED12 -> 1_LED13
- J12 pad 9: 1_RE12_A -> 1_RE12_B
- J14 pad 15: 1_RE8_B -> 1_RE8_A
- J14 pad 16: 1_RE8_A -> 1_RE8_B
- J14 pad 18: 1_RE7_B -> 1_RE7_A
- J14 pad 19: 1_RE7_A -> 1_RE7_B
- J14 pad 21: 1_RE6_B -> 1_RE6_A
- J14 pad 22: 1_RE6_A -> 1_RE6_B
- R110 pad 1: 0_FPGA_DONE -> 1_FPGA_DONE
Routing:
- net Net-(D69-K): track 2.14 -> 83.8 mm, vias 0 -> 16
- net Net-(D53-K): track 2.14 -> 83.8 mm, vias 0 -> 16
- net Net-(D245-K): track 2.14 -> 83.8 mm, vias 0 -> 16
- net Net-(D229-K): track 2.14 -> 83.8 mm, vias 0 -> 16
- net Net-(D213-K): track 2.14 -> 83.8 mm, vias 0 -> 16
- net Net-(D197-K): track 2.14 -> 83.8 mm, vias 0 -> 16
- net Net-(D181-K): track 2.14 -> 83.8 mm, vias 0 -> 16
- net Net-(D165-K): track 2.14 -> 83.8 mm, vias 0 -> 16
- net Net-(D149-K): track 2.14 -> 83.8 mm, vias 0 -> 16
- net Net-(D133-K): track 2.14 -> 83.8 mm, vias 0 -> 16
- net Net-(D117-K): track 2.14 -> 83.8 mm, vias 0 -> 16
- net Net-(D101-K): track 2.14 -> 83.8 mm, vias 0 -> 16
- net Net-(D100-K): track 2.14 -> 83.8 mm, vias 0 -> 16
- net Net-(D37-K): track 2.14 -> 83.8 mm, vias 0 -> 16
- net Net-(D21-K): track 2.14 -> 83.8 mm, vias 0 -> 16
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- added copper zone on In2.Cu, net DVCC_3V3
- added copper zone on In3.Cu, net GND
