File: SIGMAGE_HW/SIGMAGE/SIGMAGE.kicad_pcb (KiCad board)
At the start: 6 copper layers, 270 x 170 mm, 719 parts, among them J1 UJ31CHG2SMTTR, J10 SJ63073E, J11 SJ63073E, J12 61306421821, J13 61306421121, J14 61306421821, J18 HTSW10107GD, J19 HTSW10107GD, J2 SJ63073E, J20 SJ63073E, J21 SJ63073E, J22 HTSW10107GD, J23 HTSW10107GD, J24 SJ63073E, J25 SJ63073E, J26 HTSW10107GD, J27 HTSW10107GD, J3 TSW10607GS, J4 SJ63073E, J5 TSW10607GS, J6 TSW10607GS, J7 473521001, J8 61306421121, J9 TSW10607GS, U1 MAX8902BATA/V+T, U10 PCM5102APWR, U11 TPS62130RGTT, U12 TPS62130RGTT, U13 ESDR0502NMUTBG, U14 93LC56-I/SN, U15 STM32F407VGTx, U16 OPA1612AIDRGR, U17 OPA1612AIDRGR, U18 PCM1803ADB, U19 PCM1803ADB, U2 MAX8902BATA/V+T, U20 PCM5102APWR, U21 PCM5102APWR, U22 EC11E183440C, U23 EC11E183440C, U24 EC11E183440C, U25 EC11E183440C, U26 EC11E183440C, U27 EC11E183440C, U28 EC11E183440C, U29 EC11E183440C, U3 PCM5102APWR, U30 EC11E183440C, U31 MAX8902BATA/V+T, U32 EC11E183440C, U33 EC11E183440C, U34 EC11E183440C, U35 EC11E183440C, U36 EC11E183440C, U37 EC11E183440C, U4 OPA1612AIDRGR, U41 MMBT2222A, U42 TPS62130RGTT, U5 PCM1803ADB, U6 OPA1612AIDRGR, U7 PCM1803ADB, U8 LFE5U25F6BG256I, U9 FT2232HLTRAY, X1 STDCSU18M

Commit message: improvements
Parts:
- added R186: 33, Resistor_SMD:R_0603_1608Metric, F.Cu at (97.5, 159.8)
- added R187: 33, Resistor_SMD:R_0603_1608Metric, F.Cu at (97.5, 158.2)
- added R188: 33, Resistor_SMD:R_0603_1608Metric, F.Cu at (97.5, 156.8)
- added R189: 33, Resistor_SMD:R_0603_1608Metric, F.Cu at (122.5, 159.8)
- added R190: 33, Resistor_SMD:R_0603_1608Metric, F.Cu at (122.5, 158.2)
- added R191: 33, Resistor_SMD:R_0603_1608Metric, F.Cu at (122.5, 156.8)
- C12, C125, C126, C127, C128, C129, C13, C130, C131, C132, C133, C134, C135, C136, C137, C138, C139, C140, C141, C142, C165, C166, C167, C168, C173, C174, C175, C176, C179, C18, C180, C181, C182, C183, C184, C185, C186, C19, C20, C21, C22, C23, C62, C63, C82, C83, C89, C90: footprint Resistor_SMD:R_0603_1608Metric -> Capacitor_SMD:C_0603_1608Metric
- moved C153 15.3 mm to (146.2, 175.8), turned to 0 degrees
- moved C155 15.3 mm to (146.2, 201.8), turned to 0 degrees
- moved C58 15.3 mm to (146.2, 123.8), turned to 0 degrees
- moved C76 15.3 mm to (146.2, 149.8), turned to 0 degrees
- moved C157 13.2 mm to (146.2, 174.2), turned to 0 degrees
- moved C159 13.2 mm to (146.2, 200.2), turned to 0 degrees
- moved C59 13.2 mm to (146.2, 122.2), turned to 0 degrees
- moved C78 13.2 mm to (146.2, 148.2), turned to 0 degrees
- moved C154 11.8 mm to (150.0, 173.5), turned to -90 degrees
- moved C156 11.8 mm to (150.0, 199.5), turned to -90 degrees
- moved C60 11.8 mm to (150.0, 121.5), turned to -90 degrees
- moved C77 11.8 mm to (150.0, 147.5), turned to -90 degrees
- moved C148 11.7 mm to (140.8, 188.8), turned to 180 degrees
- moved C66 11.7 mm to (140.8, 110.8), turned to 180 degrees
- moved C73 11.7 mm to (140.8, 136.8), turned to 180 degrees
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Connections:
- net 0_DAC1_SD renamed 0_DAC1_DIN
- net 0_DAC2_SD renamed 0_DAC2_DIN
- net 0_DAC3_SD renamed 0_DAC3_DIN
- net 0_DAC4_SD renamed 0_DAC4_DIN
- U10 pad 10: 0_DAC2_DEMP -> GND
- U10 pad 12: 0_DAC2_SCK -> 0_BUS_DAC_SCK
- U10 pad 13: 0_DAC2_CK -> 0_BUS_DAC_BCK
- U10 pad 15: 0_DAC2_WS -> 0_BUS_DAC_LRCK
- U10 pad 16: 0_DAC2_FMT -> GND
- U18 pad 10: 0_ADC3_LRCK -> 0_BUS_ADC_LRCK
- U18 pad 11: 0_ADC3_BCK -> 0_BUS_ADC_BCK
- U18 pad 15: 0_ADC3_SCKI -> 0_BUS_ADC_SCK
- U18 pad 17: 0_ADC3_FMT0 -> DVCC_3V3
- U18 pad 18: 0_ADC3_FMT1 -> GND
- U18 pad 19: 0_ADC3_MODE0 -> GND
- U18 pad 20: 0_ADC3_MODE1 -> GND
- U19 pad 10: 0_ADC4_LRCK -> 0_BUS_ADC_LRCK
- U19 pad 11: 0_ADC4_BCK -> 0_BUS_ADC_BCK
- U19 pad 15: 0_ADC4_SCKI -> 0_BUS_ADC_SCK
- U19 pad 17: 0_ADC4_FMT0 -> DVCC_3V3
- U19 pad 18: 0_ADC4_FMT1 -> GND
- U19 pad 19: 0_ADC4_MODE0 -> GND
- U19 pad 20: 0_ADC4_MODE1 -> GND
- U20 pad 10: 0_DAC3_DEMP -> GND
- U20 pad 12: 0_DAC3_SCK -> 0_BUS_DAC_SCK
- U20 pad 13: 0_DAC3_CK -> 0_BUS_DAC_BCK
- U20 pad 15: 0_DAC3_WS -> 0_BUS_DAC_LRCK
- U20 pad 16: 0_DAC3_FMT -> GND
- U21 pad 10: 0_DAC4_DEMP -> GND
- U21 pad 12: 0_DAC4_SCK -> 0_BUS_DAC_SCK
- U21 pad 13: 0_DAC4_CK -> 0_BUS_DAC_BCK
- U21 pad 15: 0_DAC4_WS -> 0_BUS_DAC_LRCK
- U21 pad 16: 0_DAC4_FMT -> GND
- U3 pad 10: 0_DAC1_DEMP -> GND
- U3 pad 12: 0_DAC1_SCK -> 0_BUS_DAC_SCK
- U3 pad 13: 0_DAC1_CK -> 0_BUS_DAC_BCK
- U3 pad 15: 0_DAC1_WS -> 0_BUS_DAC_LRCK
- U3 pad 16: 0_DAC1_FMT -> GND
- U5 pad 10: 0_ADC1_LRCK -> 0_BUS_ADC_LRCK
- U5 pad 11: 0_ADC1_BCK -> 0_BUS_ADC_BCK
- U5 pad 15: 0_ADC1_SCKI -> 0_BUS_ADC_SCK
- U5 pad 17: 0_ADC1_FMT0 -> DVCC_3V3
- U5 pad 18: 0_ADC1_FMT1 -> GND
- U5 pad 19: 0_ADC1_MODE0 -> GND
- U5 pad 20: 0_ADC1_MODE1 -> GND
- U7 pad 10: 0_ADC2_LRCK -> 0_BUS_ADC_LRCK
- U7 pad 11: 0_ADC2_BCK -> 0_BUS_ADC_BCK
- U7 pad 15: 0_ADC2_SCKI -> 0_BUS_ADC_SCK
- U7 pad 17: 0_ADC2_FMT0 -> DVCC_3V3
- U7 pad 18: 0_ADC2_FMT1 -> GND
- U7 pad 19: 0_ADC2_MODE0 -> GND
- U7 pad 20: 0_ADC2_MODE1 -> GND
- U8 pad C16: unconnected-(U8D-PR5A-PadC16) -> 0_ADC4_OSR
- U8 pad D16: unconnected-(U8D-PR8A-PadD16) -> 0_ADC4_DOUT
- U8 pad E15: unconnected-(U8D-PR8B-PadE15) -> 0_ADC4_PYPAS
- U8 pad E16: unconnected-(U8D-PR11D-PadE16) -> 0_ADC4_PDWN
- U8 pad F15: unconnected-(U8D-PR11C-PadF15) -> 0_ADC3_OSR
- U8 pad F16: unconnected-(U8D-PR14A-PadF16) -> 0_ADC3_DOUT
- U8 pad G15: unconnected-(U8D-PR14B-PadG15) -> 0_ADC3_PYPAS
- U8 pad G16: unconnected-(U8D-PR20A-PadG16) -> 0_ADC3_PDWN
- U8 pad H15: unconnected-(U8D-PR20B-PadH15) -> 0_ADC_SCK
- U8 pad H2: unconnected-(U8H-PL20B-PadH2) -> 0_DAC_SCK
- U8 pad J1: unconnected-(U8H-PL23A-PadJ1) -> 0_DAC_BCK
- U8 pad J15: unconnected-(U8D-PR23B-PadJ15) -> 0_ADC_LRCK
- U8 pad J16: unconnected-(U8D-PR23A-PadJ16) -> 0_ADC_BCK
- U8 pad J2: unconnected-(U8H-PL23B-PadJ2) -> 0_DAC_LRCK
- U8 pad K15: unconnected-(U8D-PR23D-PadK15) -> 0_ADC2_DOUT
- U8 pad K16: unconnected-(U8D-PR23C-PadK16) -> 0_ADC2_OSR
- U8 pad L15: unconnected-(U8E-PR26B-PadL15) -> 0_ADC2_PDWN
- U8 pad L16: unconnected-(U8E-PR26A-PadL16) -> 0_ADC2_PYPAS
- U8 pad M15: unconnected-(U8E-PR26D-PadM15) -> 0_ADC1_DOUT
- U8 pad M16: unconnected-(U8E-PR26C-PadM16) -> 0_ADC1_OSR
- U8 pad N16: unconnected-(U8E-PR32A-PadN16) -> 0_ADC1_PYPAS
- U8 pad P16: unconnected-(U8E-PR35A-PadP16) -> 0_ADC1_PDWN
Routing:
- net 0_BUS_ADC_LRCK: track 0.00 -> 153.0 mm, vias 0 -> 5
- net 0_BUS_ADC_BCK: track 0.00 -> 151.9 mm, vias 0 -> 5
- net 0_BUS_ADC_SCK: track 0.00 -> 137.7 mm, vias 0 -> 5
- net 0_BUS_DAC_LRCK: track 0.00 -> 134.4 mm, vias 0 -> 5
- net 0_BUS_DAC_BCK: track 0.00 -> 128.2 mm, vias 0 -> 5
- net 0_BUS_DAC_SCK: track 0.00 -> 126.4 mm, vias 0 -> 5
- net 0_ADC1_PYPAS: track 0.00 -> 61.4 mm
- net 0_ADC1_PDWN: track 0.00 -> 60.4 mm
- net 0_ADC4_DOUT: track 0.00 -> 59.5 mm
- net 0_ADC4_PYPAS: track 0.00 -> 58.8 mm
- net 0_ADC1_OSR: track 0.00 -> 57.4 mm
- net 0_ADC4_PDWN: track 0.00 -> 56.7 mm
- net 0_ADC4_OSR: track 0.00 -> 56.6 mm
- net 0_ADC1_DOUT: track 12.6 -> 62.2 mm
- net 0_ADC2_DOUT: track 0.00 -> 39.2 mm
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
Commit message: changes
Parts:
- R28, R60: value 2200 -> 4700
