File: SIGMAGE_HW/SIGMAGE/LED.kicad_sch (KiCad schematic)
At the start: 272 parts

Commit message: changes
Changed lines of the file:
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@@
+		)
+	)
+	(label "Verify FPGA GPIO's can handle 33mA"
+		(at 275.59 66.04 0)
+		(effects
+			(font
+				(size 3.81 3.81)
+				(thickness 0.508)
+				(bold yes)
+				(italic yes)
+				(color 255 0 0 1)
+			)
+			(justify left bottom)
 		)
 	)

Commit message: almost done
Parts:
- R100, R101, R102, R103, R104, R105, R106, R91, R92, R93, R94, R95, R96, R97, R98, R99: value 1k -> 260
Changed lines of the file:
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@@
 		)
 	)
-	(label "Verify FPGA GPIO's can handle 33mA"
+	(label "Use LED's with 2Vfwd at 5mA"
 		(at 275.59 66.04 0)
 		(effects
@@
 			)
 		)
-		(property "Value" "1k"
-			(at 233.68 162.56 90)
+		(property "Value" "260"
+			(at 234.188 162.56 90)
 			(show_name no)
 			(do_not_autoplace no)
@@
 			)
 		)
-		(property "Value" "1k"
-			(at 233.68 172.72 90)
+		(property "Value" "260"
+			(at 234.188 172.72 90)
 			(show_name no)
 			(do_not_autoplace no)
@@
 			)
 		)
-		(property "Value" "1k"
-			(at 233.68 101.6 90)
+		(property "Value" "260"
+			(at 234.188 101.6 90)
 			(show_name no)
 			(do_not_autoplace no)
@@
 			)
 		)
-		(property "Value" "1k"
-			(at 233.68 111.76 90)
+		(property "Value" "260"
+			(at 234.188 111.76 90)
 			(show_name no)
 			(do_not_autoplace no)
@@
 			)
 		)
-		(property "Value" "1k"
-			(at 233.68 142.24 90)
+		(property "Value" "260"
+			(at 234.188 142.24 90)
 			(show_name no)
 			(do_not_autoplace no)
@@
 			)
 		)
-		(property "Value" "1k"
-			(at 233.68 60.96 90)
+		(property "Value" "260"
+			(at 234.188 60.96 90)
 			(show_name no)
 			(do_not_autoplace no)
@@
 			)
 		)
-		(property "Value" "1k"
-			(at 233.68 91.44 90)
+		(property "Value" "260"
+			(at 234.188 91.44 90)
 			(show_name no)
 			(do_not_autoplace no)
@@
 			)
 		)
-		(property "Value" "1k"
-			(at 233.68 50.8 90)
+		(property "Value" "260"
+			(at 234.188 50.8 90)
 			(show_name no)
 			(do_not_autoplace no)
@@
 			)
 		)
-		(property "Value" "1k"
-			(at 233.68 132.08 90)
+		(property "Value" "260"
+			(at 234.188 132.08 90)
 			(show_name no)
 			(do_not_autoplace no)
@@
 			)
 		)
-		(property "Value" "1k"
-			(at 233.68 193.04 90)
+		(property "Value" "260"
+			(at 234.188 193.04 90)
 			(show_name no)
 			(do_not_autoplace no)
@@
 			)
 		)
-		(property "Value" "1k"
-			(at 233.68 121.92 90)
+		(property "Value" "260"
+			(at 234.188 121.92 90)
 			(show_name no)
 			(do_not_autoplace no)
@@
 			)
 		)
-		(property "Value" "1k"
-			(at 233.68 81.28 90)
+		(property "Value" "260"
+			(at 234.188 81.28 90)
 			(show_name no)
 			(do_not_autoplace no)
@@
 			)
 		)
-		(property "Value" "1k"
-			(at 233.68 71.12 90)
+		(property "Value" "260"
+			(at 234.188 71.12 90)
 			(show_name no)
 			(do_not_autoplace no)
@@
 			)
 		)
-		(property "Value" "1k"
-			(at 233.68 203.2 90)
+		(property "Value" "260"
+			(at 234.188 203.2 90)
 			(show_name no)
 			(do_not_autoplace no)
@@
 			)
 		)
-		(property "Value" "1k"
-			(at 233.68 182.88 90)
+		(property "Value" "260"
+			(at 234.188 182.88 90)
 			(show_name no)
 			(do_not_autoplace no)
@@
 			)
 		)
-		(property "Value" "1k"
-			(at 233.68 152.4 90)
+		(property "Value" "260"
+			(at 234.188 152.4 90)
 			(show_name no)
 			(do_not_autoplace no)

Commit message: before sync sheets
Connections:
- net LED_C0 renamed T_LED_C1
- net LED_C1 renamed T_LED_C2
- net LED_C10 renamed T_LED_C11
- net LED_C11 renamed T_LED_C12
- net LED_C12 renamed T_LED_C13
- net LED_C13 renamed T_LED_C14
- net LED_C14 renamed T_LED_C15
- net LED_C15 renamed T_LED_C16
- net LED_C2 renamed T_LED_C3
- net LED_C3 renamed T_LED_C4
- net LED_C4 renamed T_LED_C5
- net LED_C5 renamed T_LED_C6
- net LED_C6 renamed T_LED_C7
- net LED_C7 renamed T_LED_C8
- net LED_C8 renamed T_LED_C9
- net LED_C9 renamed T_LED_C10
- net LED_R0 renamed T_LED_R1
- net LED_R1 renamed T_LED_R2
- net LED_R10 renamed T_LED_R11
- net LED_R11 renamed T_LED_R12
- net LED_R12 renamed T_LED_R13
- net LED_R13 renamed T_LED_R14
- net LED_R14 renamed T_LED_R15
- net LED_R15 renamed T_LED_R16
- net LED_R2 renamed T_LED_R3
- net LED_R3 renamed T_LED_R4
- net LED_R4 renamed T_LED_R5
- net LED_R5 renamed T_LED_R6
- net LED_R6 renamed T_LED_R7
- net LED_R7 renamed T_LED_R8
- net LED_R8 renamed T_LED_R9
- net LED_R9 renamed T_LED_R10

Commit message: finished schematic
Connections:
- net T_LED_C1 renamed 1_LED_C1
- net T_LED_C10 renamed 1_LED_C10
- net T_LED_C11 renamed 1_LED_C11
- net T_LED_C12 renamed 1_LED_C12
- net T_LED_C13 renamed 1_LED_C13
- net T_LED_C14 renamed 1_LED_C14
- net T_LED_C15 renamed 1_LED_C15
- net T_LED_C16 renamed 1_LED_C16
- net T_LED_C2 renamed 1_LED_C2
- net T_LED_C3 renamed 1_LED_C3
- net T_LED_C4 renamed 1_LED_C4
- net T_LED_C5 renamed 1_LED_C5
- net T_LED_C6 renamed 1_LED_C6
- net T_LED_C7 renamed 1_LED_C7
- net T_LED_C8 renamed 1_LED_C8
- net T_LED_C9 renamed 1_LED_C9
- net T_LED_R1 renamed 1_LED_R1
- net T_LED_R10 renamed 1_LED_R10
- net T_LED_R11 renamed 1_LED_R11
- net T_LED_R12 renamed 1_LED_R12
- net T_LED_R13 renamed 1_LED_R13
- net T_LED_R14 renamed 1_LED_R14
- net T_LED_R15 renamed 1_LED_R15
- net T_LED_R16 renamed 1_LED_R16
- net T_LED_R2 renamed 1_LED_R2
- net T_LED_R3 renamed 1_LED_R3
- net T_LED_R4 renamed 1_LED_R4
- net T_LED_R5 renamed 1_LED_R5
- net T_LED_R6 renamed 1_LED_R6
- net T_LED_R7 renamed 1_LED_R7
- net T_LED_R8 renamed 1_LED_R8
- net T_LED_R9 renamed 1_LED_R9
Other:
- moved on the sheet: D10, D100, D101, D102, D103, D104, D105, D106, D107, D108, D109, D11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
