File: SIGMAGE_HW/SIGMAGE/ADC.kicad_sch (KiCad schematic)
At the start: 68 parts, among them J10 SJ63073E, J11 SJ63073E, J2 SJ63073E, J4 SJ63073E, U16 OPA1612AIDRGR, U17 OPA1612AIDRGR, U18 PCM1803ADB, U19 PCM1803ADB, U4 OPA1612AIDRGR, U5 PCM1803ADB, U6 OPA1612AIDRGR, U7 PCM1803ADB

Commit message: finished schematic
Connections:
- net ADC1_BCK renamed 0_ADC1_BCK
- net ADC1_BYPAS renamed 0_ADC1_PYPAS
- net ADC1_DOUT renamed 0_ADC1_DOUT
- net ADC1_FMT0 renamed 0_ADC1_FMT0
- net ADC1_FMT1 renamed 0_ADC1_FMT1
- net ADC1_LRCK renamed 0_ADC1_LRCK
- net ADC1_MODE0 renamed 0_ADC1_MODE0
- net ADC1_MODE1 renamed 0_ADC1_MODE1
- net ADC1_OSR renamed 0_ADC1_OSR
- net ADC1_PDWN renamed 0_ADC1_PDWN
- net ADC1_SCKI renamed 0_ADC1_SCKI
- net ADC2_BCK renamed 0_ADC2_BCK
- net ADC2_BYPAS renamed 0_ADC2_PYPAS
- net ADC2_DOUT renamed 0_ADC2_DOUT
- net ADC2_FMT0 renamed 0_ADC2_FMT0
- net ADC2_FMT1 renamed 0_ADC2_FMT1
- net ADC2_LRCK renamed 0_ADC2_LRCK
- net ADC2_MODE0 renamed 0_ADC2_MODE0
- net ADC2_MODE1 renamed 0_ADC2_MODE1
- net ADC2_OSR renamed 0_ADC2_OSR
- net ADC2_PDWN renamed 0_ADC2_PDWN
- net ADC2_SCKI renamed 0_ADC2_SCKI
- net ADC3_BCK renamed 0_ADC3_BCK
- net ADC3_BYPAS renamed 0_ADC3_PYPAS
- net ADC3_DOUT renamed 0_ADC3_DOUT
- net ADC3_FMT0 renamed 0_ADC3_FMT0
- net ADC3_FMT1 renamed 0_ADC3_FMT1
- net ADC3_LRCK renamed 0_ADC3_LRCK
- net ADC3_MODE0 renamed 0_ADC3_MODE0
- net ADC3_MODE1 renamed 0_ADC3_MODE1
- net ADC3_OSR renamed 0_ADC3_OSR
- net ADC3_PDWN renamed 0_ADC3_PDWN
- net ADC3_SCKI renamed 0_ADC3_SCKI
- net ADC4_BCK renamed 0_ADC4_BCK
- net ADC4_BYPAS renamed 0_ADC4_PYPAS
- net ADC4_DOUT renamed 0_ADC4_DOUT
- net ADC4_FMT0 renamed 0_ADC4_FMT0
- net ADC4_FMT1 renamed 0_ADC4_FMT1
- net ADC4_LRCK renamed 0_ADC4_LRCK
- net ADC4_MODE0 renamed 0_ADC4_MODE0
- net ADC4_MODE1 renamed 0_ADC4_MODE1
- net ADC4_OSR renamed 0_ADC4_OSR
- net ADC4_PDWN renamed 0_ADC4_PDWN
- net ADC4_SCKI renamed 0_ADC4_SCKI
- net AN_IN1_L renamed 0_AN_IN1_L
- net AN_IN1_R renamed 0_AN_IN1_R
- net AN_IN2_L renamed 0_AN_IN2_L
- net AN_IN2_R renamed 0_AN_IN2_R
- net AN_IN3_L renamed 0_AN_IN3_L
- net AN_IN3_R renamed 0_AN_IN3_R
- net AN_IN4_L renamed 0_AN_IN4_L
- net AN_IN4_R renamed 0_AN_IN4_R

Commit message: uga uga
Parts:
- C12, C125, C126, C127, C128, C129, C13, C130, C131, C132, C133, C134, C135, C136, C137, C138, C139, C140, C141, C142, C173, C174, C175, C176, C179, C18, C180, C181, C182, C183, C184, C185, C186, C19, C20, C21, C22, C23, C89, C90: footprint Capacitor_SMD:C_1206_3216Metric -> Resistor_SMD:R_0603_1608Metric
Changed lines of the file:
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@@
 			)
 		)
-		(property "Footprint" "Capacitor_SMD:C_1206_3216Metric"
+		(property "Footprint" "Resistor_SMD:R_0603_1608Metric"
 			(at 157.48 161.5948 0)
 			(hide yes)
@@
 			)
 		)
-		(property "Footprint" "Capacitor_SMD:C_1206_3216Metric"
+		(property "Footprint" "Resistor_SMD:R_0603_1608Metric"
 			(at 199.0852 261.62 0)
 			(hide yes)
@@
 			)
 		)
-		(property "Footprint" "Capacitor_SMD:C_1206_3216Metric"
+		(property "Footprint" "Resistor_SMD:R_0603_1608Metric"
 			(at 157.48 188.2648 0)
 			(hide yes)
@@
 			)
 		)
-		(property "Footprint" "Capacitor_SMD:C_1206_3216Metric"
+		(property "Footprint" "Resistor_SMD:R_0603_1608Metric"
 			(at 416.2552 121.92 0)
 			(hide yes)
@@
 			)
 		)
-		(property "Footprint" "Capacitor_SMD:C_1206_3216Metric"
+		(property "Footprint" "Resistor_SMD:R_0603_1608Metric"
 			(at 383.2352 299.72 0)
 			(hide yes)
@@
 			)
 		)
-		(property "Footprint" "Capacitor_SMD:C_1206_3216Metric"
+		(property "Footprint" "Resistor_SMD:R_0603_1608Metric"
 			(at 370.5352 77.47 0)
 			(hide yes)
@@
 			)
 		)
-		(property "Footprint" "Capacitor_SMD:C_1206_3216Metric"
+		(property "Footprint" "Resistor_SMD:R_0603_1608Metric"
 			(at 157.48 87.9348 0)
 			(hide yes)
@@
 			)
 		)
-		(property "Footprint" "Capacitor_SMD:C_1206_3216Metric"
+		(property "Footprint" "Resistor_SMD:R_0603_1608Metric"
 			(at 383.2352 224.79 0)
 			(hide yes)
@@
 			)
 		)
-		(property "Footprint" "Capacitor_SMD:C_1206_3216Metric"
+		(property "Footprint" "Resistor_SMD:R_0603_1608Metric"
 			(at 309.5752 83.82 0)
 			(hide yes)
@@
 			)
 		)
-		(property "Footprint" "Capacitor_SMD:C_1206_3216Metric"
+		(property "Footprint" "Resistor_SMD:R_0603_1608Metric"
 			(at 403.5552 121.92 0)
 			(hide yes)
@@
 			)
 		)
-		(property "Footprint" "Capacitor_SMD:C_1206_3216Metric"
+		(property "Footprint" "Resistor_SMD:R_0603_1608Metric"
 			(at 403.5552 195.58 0)
 			(hide yes)
@@
 			)
 		)
-		(property "Footprint" "Capacitor_SMD:C_1206_3216Metric"
+		(property "Footprint" "Resistor_SMD:R_0603_1608Metric"
 			(at 309.5752 231.14 0)
 			(hide yes)
@@
 			)
 		)
-		(property "Footprint" "Capacitor_SMD:C_1206_3216Metric"
+		(property "Footprint" "Resistor_SMD:R_0603_1608Metric"
 			(at 403.5552 344.17 0)
 			(hide yes)
@@
 			)
 		)
-		(property "Footprint" "Capacitor_SMD:C_1206_3216Metric"
+		(property "Footprint" "Resistor_SMD:R_0603_1608Metric"
 			(at 321.0052 157.48 0)
 			(hide yes)
@@
 			)
 		)
-		(property "Footprint" "Capacitor_SMD:C_1206_3216Metric"
+		(property "Footprint" "Resistor_SMD:R_0603_1608Metric"
 			(at 199.0852 87.63 0)
 			(hide yes)
@@
 			)
 		)
-		(property "Footprint" "Capacitor_SMD:C_1206_3216Metric"
+		(property "Footprint" "Resistor_SMD:R_0603_1608Metric"
 			(at 321.0052 83.82 0)
 			(hide yes)
@@
 			)
 		)
-		(property "Footprint" "Capacitor_SMD:C_1206_3216Metric"
+		(property "Footprint" "Resistor_SMD:R_0603_1608Metric"
 			(at 157.48 114.6048 0)
 			(hide yes)
@@
 			)
 		)
-		(property "Footprint" "Capacitor_SMD:C_1206_3216Metric"
+		(property "Footprint" "Resistor_SMD:R_0603_1608Metric"
 			(at 370.5352 151.13 0)
 			(hide yes)
@@
 			)
 		)
-		(property "Footprint" "Capacitor_SMD:C_1206_3216Metric"
+		(property "Footprint" "Resistor_SMD:R_0603_1608Metric"
 			(at 370.5352 299.72 0)
 			(hide yes)
@@
 			)
 		)
-		(property "Footprint" "Capacitor_SMD:C_1206_3216Metric"
+		(property "Footprint" "Resistor_SMD:R_0603_1608Metric"
 			(at 416.2552 344.17 0)
 			(hide yes)
@@
 			)
 		)
-		(property "Footprint" "Capacitor_SMD:C_1206_3216Metric"
+		(property "Footprint" "Resistor_SMD:R_0603_1608Metric"
 			(at 199.0852 161.29 0)
 			(hide yes)
@@
 			)
 		)
-		(property "Footprint" "Capacitor_SMD:C_1206_3216Metric"
+		(property "Footprint" "Resistor_SMD:R_0603_1608Metric"
 			(at 370.5352 224.79 0)
 			(hide yes)
@@
 			)
 		)
-		(property "Footprint" "Capacitor_SMD:C_1206_3216Metric"
+		(property "Footprint" "Resistor_SMD:R_0603_1608Metric"
 			(at 416.2552 269.24 0)
 			(hide yes)
@@
 			)
 		)
-		(property "Footprint" "Capacitor_SMD:C_1206_3216Metric"
+		(property "Footprint" "Resistor_SMD:R_0603_1608Metric"
 			(at 199.0852 187.96 0)
 			(hide yes)
@@
 			)
 		)
-		(property "Footprint" "Capacitor_SMD:C_1206_3216Metric"
+		(property "Footprint" "Resistor_SMD:R_0603_1608Metric"
 			(at 321.0052 231.14 0)
 			(hide yes)
@@
 			)
 		)
-		(property "Footprint" "Capacitor_SMD:C_1206_3216Metric"
+		(property "Footprint" "Resistor_SMD:R_0603_1608Metric"
 			(at 309.5752 306.07 0)
 			(hide yes)
@@
 			)
 		)
-		(property "Footprint" "Capacitor_SMD:C_1206_3216Metric"
+		(property "Footprint" "Resistor_SMD:R_0603_1608Metric"
 			(at 157.48 261.9248 0)
 			(hide yes)
@@
 			)
 		)
-		(property "Footprint" "Capacitor_SMD:C_1206_3216Metric"
+		(property "Footprint" "Resistor_SMD:R_0603_1608Metric"
 			(at 199.0852 336.55 0)
 			(hide yes)
@@
 			)
 		)
-		(property "Footprint" "Capacitor_SMD:C_1206_3216Metric"
+		(property "Footprint" "Resistor_SMD:R_0603_1608Metric"
 			(at 157.48 336.8548 0)
 			(hide yes)
@@
 			)
 		)
-		(property "Footprint" "Capacitor_SMD:C_1206_3216Metric"
+		(property "Footprint" "Resistor_SMD:R_0603_1608Metric"
 			(at 157.48 235.2548 0)
 			(hide yes)
@@
 			)
 		)
-		(property "Footprint" "Capacitor_SMD:C_1206_3216Metric"
+		(property "Footprint" "Resistor_SMD:R_0603_1608Metric"
 			(at 199.0852 234.95 0)
 			(hide yes)
@@
 			)
 		)
-		(property "Footprint" "Capacitor_SMD:C_1206_3216Metric"
+		(property "Footprint" "Resistor_SMD:R_0603_1608Metric"
 			(at 383.2352 151.13 0)
 			(hide yes)
@@
 			)
 		)
-		(property "Footprint" "Capacitor_SMD:C_1206_3216Metric"
+		(property "Footprint" "Resistor_SMD:R_0603_1608Metric"
 			(at 199.0852 309.88 0)
 			(hide yes)
@@
 			)
 		)
-		(property "Footprint" "Capacitor_SMD:C_1206_3216Metric"
+		(property "Footprint" "Resistor_SMD:R_0603_1608Metric"
 			(at 309.5752 157.48 0)
 			(hide yes)
@@
 			)
 		)
-		(property "Footprint" "Capacitor_SMD:C_1206_3216Metric"
+		(property "Footprint" "Resistor_SMD:R_0603_1608Metric"
 			(at 416.2552 195.58 0)
 			(hide yes)
@@
 			)
 		)
-		(property "Footprint" "Capacitor_SMD:C_1206_3216Metric"
+		(property "Footprint" "Resistor_SMD:R_0603_1608Metric"
 			(at 383.2352 77.47 0)
 			(hide yes)
@@
 			)
 		)
-		(property "Footprint" "Capacitor_SMD:C_1206_3216Metric"
+		(property "Footprint" "Resistor_SMD:R_0603_1608Metric"
 			(at 321.0052 306.07 0)
 			(hide yes)
@@
 			)
 		)
-		(property "Footprint" "Capacitor_SMD:C_1206_3216Metric"
+		(property "Footprint" "Resistor_SMD:R_0603_1608Metric"
 			(at 157.48 310.1848 0)
 			(hide yes)
@@
 			)
 		)
-		(property "Footprint" "Capacitor_SMD:C_1206_3216Metric"
+		(property "Footprint" "Resistor_SMD:R_0603_1608Metric"
 			(at 199.0852 114.3 0)
 			(hide yes)
@@
 			)
 		)
-		(property "Footprint" "Capacitor_SMD:C_1206_3216Metric"
+		(property "Footprint" "Resistor_SMD:R_0603_1608Metric"
 			(at 403.5552 269.24 0)
 			(hide yes)
