File: SIGMAGE_HW/SIGMAGE/BTN.kicad_sch (KiCad schematic)
At the start: 0 parts

Commit message: changes
Parts:
- added C17, C193, C194, C195, C196, C197, C198, C199, C24, C25, C26, C27: 100n, Capacitor_SMD:C_0603_1608Metric, symbol Device:C
- added R157, R158, R159, R160, R161, R162, R163, R164, R165, R166, R167, R168: 10k, Resistor_SMD:R_0603_1608Metric, symbol Device:R
- added S1, S10, S11, S12, S2, S3, S4, S5, S6, S7, S8, S9: TL2201EEYA, SIGMAGE:TL2201EEYA, symbol SIGMAGE:TL2201EEYA
Connections:
- new net DVCC_3V3: R157.2, R158.2, R159.2, R160.2, R161.2, R162.2, R163.2, R164.2, R165.2, R166.2, R167.2, R168.2
- new net GND: C17.2, C193.2, C194.2, C195.2, C196.2, C197.2, C198.2, C199.2, C24.2, C25.2, C26.2, C27.2, S1.3 (NO_1), S10.3 (NO_1), S11.3 (NO_1), S12.3 (NO_1), S2.3 (NO_1), S3.3 (NO_1), S4.3 (NO_1), S5.3 (NO_1), S6.3 (NO_1), S7.3 (NO_1), S8.3 (NO_1), S9.3 (NO_1)
- new net SW1: C17.1, R157.1, S1.2 (COM_1)
- new net SW10: C197.1, R166.1, S10.2 (COM_1)
- new net SW11: C198.1, R167.1, S11.2 (COM_1)
- new net SW12: C199.1, R168.1, S12.2 (COM_1)
- new net SW2: C24.1, R158.1, S2.2 (COM_1)
- new net SW3: C25.1, R159.1, S3.2 (COM_1)
- new net SW4: C26.1, R160.1, S4.2 (COM_1)
- new net SW5: C27.1, R161.1, S5.2 (COM_1)
- new net SW6: C193.1, R162.1, S6.2 (COM_1)
- new net SW7: C194.1, R163.1, S7.2 (COM_1)
- new net SW8: C195.1, R164.1, S8.2 (COM_1)
- new net SW9: C196.1, R165.1, S9.2 (COM_1)
- no-connect marks 0 -> 48

Commit message: finished schematic
Connections:
- net SW1 renamed 1_SW1
- net SW10 renamed 1_SW10
- net SW11 renamed 1_SW11
- net SW12 renamed 1_SW12
- net SW2 renamed 1_SW2
- net SW3 renamed 1_SW3
- net SW4 renamed 1_SW4
- net SW5 renamed 1_SW5
- net SW6 renamed 1_SW6
- net SW7 renamed 1_SW7
- net SW8 renamed 1_SW8
- net SW9 renamed 1_SW9

Commit message: uga uga
Parts:
- removed C193, C194, C195, C196, C197, C198, C199: 100n, Capacitor_SMD:C_0603_1608Metric, symbol Device:C
- removed R162, R163, R164, R165, R166, R167, R168: 10k, Resistor_SMD:R_0603_1608Metric, symbol Device:R
- removed S10, S11, S12, S6, S7, S8, S9: TL2201EEYA, SIGMAGE:TL2201EEYA, symbol SIGMAGE:TL2201EEYA
Connections:
- no-connect marks 48 -> 20
