File: SIGMAGE_HW/SIGMAGE/ENC.kicad_sch (KiCad schematic)
At the start: 0 parts

Commit message: major changes
Parts:
- added R67, R68, R69, R70, R71, R72, R73, R74, R75, R76, R77, R78, R79, R80, R81, R82, R83, R84, R85, R86, R87, R88, R89, R90: 10k, Resistor_SMD:R_0603_1608Metric, symbol Device:R
- added U22, U23, U24, U25, U26, U27, U28, U29: EC11E183440C, SIGMAGE:EC11E183440C, symbol SIGMAGE:EC11E183440C
Connections:
- new net DVCC_3V3: R67.2, R68.2, R69.2, R70.2, R71.2, R72.2, R73.2, R74.2, R75.2, R76.2, R77.2, R78.2, R79.2, R80.2, R81.2, R82.2, R83.2, R84.2, R85.2, R86.2, R87.2, R88.2, R89.2, R90.2
- new net GND: U22.C1, U22.E1, U22.MH1, U22.MH2, U23.C1, U23.E1, U23.MH1, U23.MH2, U24.C1, U24.E1, U24.MH1, U24.MH2, U25.C1, U25.E1, U25.MH1, U25.MH2, U26.C1, U26.E1, U26.MH1, U26.MH2, U27.C1, U27.E1, U27.MH1, U27.MH2, U28.C1, U28.E1, U28.MH1, U28.MH2, U29.C1, U29.E1, U29.MH1, U29.MH2
- new net RE1_A: R67.1, U22.A1
- new net RE1_B: R68.1, U22.B1
- new net RE1_C: R69.1, U22.D1
- new net RE2_A: R70.1, U23.A1
- new net RE2_B: R72.1, U23.B1
- new net RE2_C: R71.1, U23.D1
- new net RE3_A: R73.1, U24.A1
- new net RE3_B: R75.1, U24.B1
- new net RE3_C: R74.1, U24.D1
- new net RE4_A: R76.1, U25.A1
- new net RE4_B: R78.1, U25.B1
- new net RE4_C: R77.1, U25.D1
- new net RE5_A: R79.1, U26.A1
- new net RE5_B: R81.1, U26.B1
- new net RE5_C: R80.1, U26.D1
- new net RE6_A: R82.1, U27.A1
- new net RE6_B: R84.1, U27.B1
- new net RE6_C: R83.1, U27.D1
- new net RE7_A: R85.1, U28.A1
- new net RE7_B: R87.1, U28.B1
- new net RE7_C: R86.1, U28.D1
- new net RE8_A: R88.1, U29.A1
- new net RE8_B: R90.1, U29.B1
- new net RE8_C: R89.1, U29.D1

Commit message: almost done
Parts:
- added R117, R118, R119, R120, R121, R122, R123, R124, R125, R126, R127, R128, R129, R130, R131, R132, R133, R134, R135, R136, R137, R138, R139, R140, R141, R142, R143, R144, R145, R146: 10k, Resistor_SMD:R_0603_1608Metric, symbol Device:R
- added U30, U32, U33, U34, U35, U36, U37, U38, U39, U40: EC11E183440C, SIGMAGE:EC11E183440C, symbol SIGMAGE:EC11E183440C
Connections:
- net DVCC_3V3: now also R117.2, R118.2, R119.2, R120.2, R121.2, R122.2, R123.2, R124.2, R125.2, R126.2, R127.2, R128.2, R129.2, R130.2, R131.2, R132.2, R133.2, R134.2, R135.2, R136.2, R137.2, R138.2, R139.2, R140.2, R141.2, R142.2, R143.2, R144.2, R145.2, R146.2
- net GND: now also U30.C1, U30.E1, U30.MH1, U30.MH2, U32.C1, U32.E1, U32.MH1, U32.MH2, U33.C1, U33.E1, U33.MH1, U33.MH2, U34.C1, U34.E1, U34.MH1, U34.MH2, U35.C1, U35.E1, U35.MH1, U35.MH2, U36.C1, U36.E1, U36.MH1, U36.MH2, U37.C1, U37.E1, U37.MH1, U37.MH2, U38.C1, U38.E1, U38.MH1, U38.MH2, U39.C1, U39.E1, U39.MH1, U39.MH2, U40.C1, U40.E1, U40.MH1, U40.MH2
- new net RE10_A: R120.1, U32.A1
- new net RE10_B: R122.1, U32.B1
- new net RE10_C: R121.1, U32.D1
- new net RE11_A: R123.1, U33.A1
- new net RE11_B: R125.1, U33.B1
- new net RE11_C: R124.1, U33.D1
- new net RE12_A: R126.1, U34.A1
- new net RE12_B: R128.1, U34.B1
- new net RE12_C: R127.1, U34.D1
- new net RE13_A: R129.1, U35.A1
- new net RE13_B: R131.1, U35.B1
- new net RE13_C: R130.1, U35.D1
- new net RE14_A: R132.1, U36.A1
- new net RE14_B: R134.1, U36.B1
- new net RE14_C: R133.1, U36.D1
- new net RE15_A: R135.1, U37.A1
- new net RE15_B: R137.1, U37.B1
- new net RE15_C: R136.1, U37.D1
- new net RE16_A: R138.1, U38.A1
- new net RE16_B: R140.1, U38.B1
- new net RE16_C: R139.1, U38.D1
- new net RE17_A: R141.1, U39.A1
- new net RE17_B: R143.1, U39.B1
- new net RE17_C: R142.1, U39.D1
- new net RE18_A: R144.1, U40.A1
- new net RE18_B: R146.1, U40.B1
- new net RE18_C: R145.1, U40.D1
- new net RE9_A: R117.1, U30.A1
- new net RE9_B: R119.1, U30.B1
- new net RE9_C: R118.1, U30.D1
Other:
- moved on the sheet: R67, R68, R69, R70, R71, R72, R73, R74, R75, R76, R77, R78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

Commit message: finished schematic
Connections:
- net RE10_A renamed 1_RE10_A
- net RE10_B renamed 1_RE10_B
- net RE10_C renamed 1_RE10_C
- net RE11_A renamed 1_RE11_A
- net RE11_B renamed 1_RE11_B
- net RE11_C renamed 1_RE11_C
- net RE12_A renamed 1_RE12_A
- net RE12_B renamed 1_RE12_B
- net RE12_C renamed 1_RE12_C
- net RE13_A renamed 1_RE13_A
- net RE13_B renamed 1_RE13_B
- net RE13_C renamed 1_RE13_C
- net RE14_A renamed 1_RE14_A
- net RE14_B renamed 1_RE14_B
- net RE14_C renamed 1_RE14_C
- net RE15_A renamed 1_RE15_A
- net RE15_B renamed 1_RE15_B
- net RE15_C renamed 1_RE15_C
- net RE16_A renamed 1_RE16_A
- net RE16_B renamed 1_RE16_B
- net RE16_C renamed 1_RE16_C
- net RE17_A renamed 1_RE17_A
- net RE17_B renamed 1_RE17_B
- net RE17_C renamed 1_RE17_C
- net RE18_A renamed 1_RE18_A
- net RE18_B renamed 1_RE18_B
- net RE18_C renamed 1_RE18_C
- net RE1_A renamed 1_RE1_A
- net RE1_B renamed 1_RE1_B
- net RE1_C renamed 1_RE1_C
- net RE2_A renamed 1_RE2_A
- net RE2_B renamed 1_RE2_B
- net RE2_C renamed 1_RE2_C
- net RE3_A renamed 1_RE3_A
- net RE3_B renamed 1_RE3_B
- net RE3_C renamed 1_RE3_C
- net RE4_A renamed 1_RE4_A
- net RE4_B renamed 1_RE4_B
- net RE4_C renamed 1_RE4_C
- net RE5_A renamed 1_RE5_A
- net RE5_B renamed 1_RE5_B
- net RE5_C renamed 1_RE5_C
- net RE6_A renamed 1_RE6_A
- net RE6_B renamed 1_RE6_B
- net RE6_C renamed 1_RE6_C
- net RE7_A renamed 1_RE7_A
- net RE7_B renamed 1_RE7_B
- net RE7_C renamed 1_RE7_C
- net RE8_A renamed 1_RE8_A
- net RE8_B renamed 1_RE8_B
- net RE8_C renamed 1_RE8_C
- net RE9_A renamed 1_RE9_A
- net RE9_B renamed 1_RE9_B
- net RE9_C renamed 1_RE9_C
Other:
- moved on the sheet: R120, R121, R122, R123, R124, R125, R126, R127, R128, R129, R130, R131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

Commit message: uga uga
Parts:
- removed R138, R139, R140, R141, R142, R143, R144, R145, R146: 10k, Resistor_SMD:R_0603_1608Metric, symbol Device:R
- removed U38, U39, U40: EC11E183440C, SIGMAGE:EC11E183440C, symbol SIGMAGE:EC11E183440C
