File: SIGMAGE_HW/SIGMAGE/PWR.kicad_sch (KiCad schematic)
At the start: 0 parts

Commit message: some USB interface
Parts:
- added C1, C29, C3, C4, C6, C7: 10u, Capacitor_SMD:C_0603_1608Metric, symbol Device:C
- added C2, C5: 10n, Capacitor_SMD:C_0603_1608Metric, symbol Device:C
- added C28, C32: 22u, Capacitor_SMD:C_0603_1608Metric, symbol Device:C
- added C30, C8: 100n, Capacitor_SMD:C_0603_1608Metric, symbol Device:C
- added C31, C9: 3300p, Capacitor_SMD:C_0603_1608Metric, symbol Device:C
- added C56, C57, C86, C87: 1u, Capacitor_SMD:C_0603_1608Metric, symbol Device:C
- added FB1, FB2, FB3, FB5: 500 @ 100 MHz, Capacitor_SMD:C_0603_1608Metric, symbol Device:FerriteBead
- added J18, J19, J22, J23: HTSW10107GD, SIGMAGE:HTSW10107GD, symbol SIGMAGE:HTSW10107GD
- added L1, L2: 2200n XFL4020-222MEB, symbol Device:L
- added R1, R2: 270k, Resistor_SMD:R_0603_1608Metric, symbol Device:R
- added R21, R25, R32, R9: 120k, Resistor_SMD:R_0603_1608Metric, symbol Device:R
- added R23, R7: 100k, Resistor_SMD:R_0603_1608Metric, symbol Device:R
- added R24: 60k, Resistor_SMD:R_0603_1608Metric, symbol Device:R
- added R4: 180k, Resistor_SMD:R_0603_1608Metric, symbol Device:R
- added R5: 200k, Resistor_SMD:R_0603_1608Metric, symbol Device:R
- added R8: 375k, Resistor_SMD:R_0603_1608Metric, symbol Device:R
- added U1, U2: MAX8902BATA/V+T, SIGMAGE:MAX8902BATAVT, symbol SIGMAGE:MAX8902BATAVT
- added U11, U12: TPS62130RGTT, SIGMAGE:TPS62130RGTT, symbol SIGMAGE:TPS62130RGTT
Connections:
- new net: L2.1, U12.1 (SW), U12.2 (SW), U12.3 (SW)
- new net: C32.1, FB5.1, L2.2, R23.1, R24.1, U12.14 (VOS)
- new net: R23.2, U12.4 (PG)
- new net: R24.2, R25.1, U12.5 (FB)
- new net: C31.1, U12.9 (SS/TR)
- new net: C5.1, C6.1, FB2.1, R4.1, U2.8 (OUT)
- new net: R4.2, R5.1
- new net: C2.1, C3.1, FB1.1, R1.1, U1.8 (OUT)
- new net: C2.2, U1.7 (BYP)
- new net: C87.1, FB5.2, J23.2
- new net: C9.1, U11.9 (SS/TR)
- new net: L1.1, U11.1 (SW), U11.2 (SW), U11.3 (SW)
- new net: C28.1, FB3.1, L1.2, R7.1, R8.1, U11.14 (VOS)
- new net: R7.2, U11.4 (PG)
- new net: R21.1, R8.2, U11.5 (FB)
- new net: C5.2, U2.7 (BYP)
- new net: C86.1, FB3.2, J22.2
- new net: R1.2, R2.1
- new net: R2.2, R9.1, U1.6 (FB)
- new net: C56.1, FB1.2, J18.2
- new net: R32.1, R5.2, U2.6 (FB)
- new net: C57.1, FB2.2, J19.2
- new net AVCC_2V5: J19.1
- new net AVCC_3V3: J18.1
- new net DVCC_1V2: J23.1
- new net DVCC_3V3: J22.1
- new net GND: C1.2, C28.2, C29.2, C3.2, C30.2, C31.2, C32.2, C4.2, C56.2, C57.2, C6.2, C7.2, C8.2, C86.2, C87.2, C9.2, R21.2, R25.2, R32.2, R9.2, U1.2 (GND), U1.4 (GS), U1.9 (EPAD), U11.15 (PGND), U11.16 (PGND), U11.17 (EPAD), U11.6 (AGND), U11.7 (FSW), U11.8 (DEF), U12.15 (PGND), U12.16 (PGND), U12.17 (EPAD), U12.6 (AGND), U12.7 (FSW), U12.8 (DEF), U2.2 (GND), U2.4 (GS), U2.9 (EPAD)
- new net VCC_5V: C1.1, C29.1, C30.1, C4.1, C7.1, C8.1, U1.1 (IN), U1.3 (EN), U11.10 (AVIN), U11.11 (PVIN), U11.12 (PVIN), U11.13 (EN), U12.10 (AVIN), U12.11 (PVIN), U12.12 (PVIN), U12.13 (EN), U2.1 (IN), U2.3 (EN)
- no-connect marks 0 -> 2

Commit message: major changes
Changed lines of the file:
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@@
 	)
 	(label "Digital Supply Reference"
-		(at 138.43 149.86 0)
+		(at 138.43 154.94 0)
 		(effects
 			(font
@@
 	)
 	(label "Analog Supply Reference"
-		(at 138.43 35.56 0)
+		(at 138.43 40.64 0)
 		(effects
 			(font

Commit message: almost done
Parts:
- added C14, C144, C16: 10u, Capacitor_SMD:C_0603_1608Metric, symbol Device:C
- added C143, C188: 1u, Capacitor_SMD:C_0603_1608Metric, symbol Device:C
- added C15: 10n, Capacitor_SMD:C_0603_1608Metric, symbol Device:C
- added C177: 100n, Capacitor_SMD:C_0603_1608Metric, symbol Device:C
- added C178: 3300p, Capacitor_SMD:C_0603_1608Metric, symbol Device:C
- added C187: 22u, Capacitor_SMD:C_0603_1608Metric, symbol Device:C
- added FB8, FB9: 500 @ 100 MHz, Capacitor_SMD:C_0603_1608Metric, symbol Device:FerriteBead
- added J26, J27: HTSW10107GD, SIGMAGE:HTSW10107GD, symbol SIGMAGE:HTSW10107GD
- added L3: 2200n XFL4020-222MEB, symbol Device:L
- added R112: 100k, Resistor_SMD:R_0603_1608Metric, symbol Device:R
- added R154: 60k, Resistor_SMD:R_0603_1608Metric, symbol Device:R
- added R155, R58: 120k, Resistor_SMD:R_0603_1608Metric, symbol Device:R
- added R3, R6: 440k, Resistor_SMD:R_0603_1608Metric, symbol Device:R
- added U31: MAX8902BATA/V+T, SIGMAGE:MAX8902BATAVT, symbol SIGMAGE:MAX8902BATAVT
- added U42: TPS62130RGTT, SIGMAGE:TPS62130RGTT, symbol SIGMAGE:TPS62130RGTT
- R24: value 60k -> 255k
Connections:
- net DVCC_1V2: now also J27.1; no longer J23.1
- net GND: now also C14.2, C143.2, C144.2, C16.2, C177.2, C178.2, C187.2, C188.2, R155.2, R58.2, U31.2 (GND), U31.4 (GS), U31.9 (EPAD), U42.15 (PGND), U42.16 (PGND), U42.17 (EPAD), U42.6 (AGND), U42.7 (FSW), U42.8 (DEF)
- net VCC_5V: now also C14.1, C144.1, C177.1, U31.1 (IN), U31.3 (EN), U42.10 (AVIN), U42.11 (PVIN), U42.12 (PVIN), U42.13 (EN)
- new net: C187.1, FB9.1, L3.2, R112.1, R154.1, U42.14 (VOS)
- new net: R154.2, R155.1, U42.5 (FB)
- new net: R3.2, R6.1
- new net: R58.1, R6.2, U31.6 (FB)
- new net: C188.1, FB9.2, J27.2
- new net: C15.1, C16.1, FB8.1, R3.1, U31.8 (OUT)
- new net: L3.1, U42.1 (SW), U42.2 (SW), U42.3 (SW)
- new net: R112.2, U42.4 (PG)
- new net: C178.1, U42.9 (SS/TR)
- new net: C143.1, FB8.2, J26.2
- new net: C15.2, U31.7 (BYP)
- new net AVCC_5V: J26.1
- new net DVCC_2V5: J23.1
- no-connect marks 2 -> 3
Other:
- moved on the sheet: C1, C2, C28, C29, C3, C30, C31, C32, C4, C5, C56, C57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

Commit message: some changes
Parts:
- removed L1, L2, L3: 2200n XFL4020-222MEB, symbol Device:L
- added L1, L2, L3: XFL4020222MEB, SIGMAGE:XFL4020222MEB, symbol SIGMAGE:XFL4020222MEB
Connections:
- net at U12.1 (SW), U12.2 (SW), U12.3 (SW): now also L2.2
- net at C32.1, FB5.1, R23.1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: now also L2.1
- net at C187.1, FB9.1, R112.1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: now also L3.1
- net at U11.1 (SW), U11.2 (SW), U11.3 (SW): now also L1.2
- net at C28.1, FB3.1, R7.1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: now also L1.1
- net at U42.1 (SW), U42.2 (SW), U42.3 (SW): now also L3.2
Other:
- moved on the sheet: C187, C188, C28, C32, C86, C87, FB3, FB5, FB9, J22, J23, J27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
