File: SIGMAGE_HW/SIGMAGE/MEZZ.kicad_sch (KiCad schematic)
At the start: 4 parts, among them J12 61306421821, J13 61306421121, J14 61306421821, J8 61306421121

Commit message: almost done with tha top part
Connections:
- net 1_LED0: now also J12.34; no longer J12.46
- net 1_LED1: now also J12.32; no longer J12.44
- net 1_LED10: now also J12.14; no longer J12.12
- net 1_LED11: now also J12.12; no longer J12.10
- net 1_LED12: now also J12.10; no longer J12.8
- net 1_LED13: now also J12.8; no longer J12.6
- net 1_LED14: now also J12.6; no longer J12.4
- net 1_LED15: now also J12.4; no longer J12.2
- net 1_LED2: now also J12.30; no longer J12.42
- net 1_LED3: now also J12.28; no longer J12.40
- net 1_LED4: now also J12.26; no longer J12.38
- net 1_LED5: now also J12.24; no longer J12.36
- net 1_LED6: now also J12.22; no longer J12.20
- net 1_LED7: now also J12.20; no longer J12.18
- net 1_LED8: now also J12.18; no longer J12.16
- net 1_LED9: now also J12.16; no longer J12.14
- net 1_RE11_A: now also J12.17; no longer J12.15
- net 1_RE11_B: now also J12.15; no longer J12.13
- net 1_RE11_C: now also J12.19; no longer J12.17
- net 1_RE12_A: now also J12.11; no longer J12.9
- net 1_RE12_B: now also J12.9; no longer J12.7
- net 1_RE12_C: now also J12.13; no longer J12.11
- net 1_RE5_A: now also J12.5; no longer J12.3
- net 1_RE5_B: now also J12.3; no longer J12.1
- net 1_RE5_C: now also J12.7; no longer J12.5
- net 1_RE6_A: now also J14.21; no longer J14.22
- net 1_RE6_B: now also J14.22; no longer J14.21
- net 1_RE7_A: now also J14.18; no longer J14.19
- net 1_RE7_B: now also J14.19; no longer J14.18
- net 1_RE8_A: now also J14.15; no longer J14.16
- net 1_RE8_B: now also J14.16; no longer J14.15
- net 1_SW1: now also J12.44; no longer J12.45
- net 1_SW2: now also J12.42; no longer J12.43
- net 1_SW3: now also J12.40; no longer J12.41
- net 1_SW4: now also J12.38; no longer J12.39
- net 1_SW5: now also J12.36; no longer J12.37
- net DVCC_3V3: now reaches J12.21
- net DVCC_3V3: now also J12.23, J12.25, J12.27, J12.29, J12.31, J12.33
- net GND: now reaches J12.35
- net GND: now also J12.37, J12.39, J12.41, J12.43, J12.45
- new net 1_FPGA_DONE: J12.2
- new net 1_FPGA_INITN: J12.1
- no-connect marks 2 -> 3
Other:
- moved on the sheet: J14, J8

Commit message: some changes
Connections:
- net DVCC_3V3: now also J14.1, J14.11, J14.13, J14.3, J14.5, J14.7, J14.9
- net GND: now also J14.10, J14.12, J14.14, J14.2, J14.4, J14.6, J14.8

Commit message: some foo
Connections:
- net 0_LED_C1: now also J13.17
- net 0_LED_C10: now also J13.26
- net 0_LED_C11: now also J13.27
- net 0_LED_C12: now also J13.28
- net 0_LED_C13: now also J13.29
- net 0_LED_C14: now also J13.30
- net 0_LED_C15: now also J13.31
- net 0_LED_C16: now also J13.32
- net 0_LED_C2: now also J13.18
- net 0_LED_C3: now also J13.19
- net 0_LED_C4: now also J13.20
- net 0_LED_C5: now also J13.21
- net 0_LED_C6: now also J13.22
- net 0_LED_C7: now also J13.23
- net 0_LED_C8: now also J13.24
- net 0_LED_C9: now also J13.25
- net 0_LED_R1: now also J13.1
- net 0_LED_R10: now also J13.10
- net 0_LED_R11: now also J13.11
- net 0_LED_R12: now also J13.12
- net 0_LED_R13: now also J13.13
- net 0_LED_R14: now also J13.14
- net 0_LED_R15: now also J13.15
- net 0_LED_R16: now also J13.16
- net 0_LED_R2: now also J13.2
- net 0_LED_R3: now also J13.3
- net 0_LED_R4: now also J13.4
- net 0_LED_R5: now also J13.5
- net 0_LED_R6: now also J13.6
- net 0_LED_R7: now also J13.7
- net 0_LED_R8: now also J13.8
- net 0_LED_R9: now also J13.9
- no-connect marks 3 -> 1

Commit message: more foo
Connections:
- net 0_FPGA_DONE: now also J8.64
- net 0_FPGA_INITN: now also J8.63
Changed lines of the file:
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@@
 		)
 	)
+	(global_label "0_FPGA_DONE"
+		(shape bidirectional)
+		(at 53.34 142.24 0)
+		(fields_autoplaced yes)
+		(effects
+			(font
+				(size 1.27 1.27)
+			)
+			(justify left)
+		)
+		(property "Intersheetrefs" "${INTERSHEET_REFS}"
+			(at 70.3784 142.24 0)
+			(hide yes)
+			(show_name no)
+			(do_not_autoplace no)
+			(effects
+				(font
+					(size 1.27 1.27)
+				)
+				(justify left)
+			)
+		)
+	)
 	(global_label "1_SW2"
 		(shape bidirectional)
@@
 		)
 	)
-	(global_label "0_FPGA_DONE"
-		(shape bidirectional)
-		(at 149.86 21.59 180)
-		(fields_autoplaced yes)
-		(effects
-			(font
-				(size 1.27 1.27)
-			)
-			(justify right)
-		)
-		(property "Intersheetrefs" "${INTERSHEET_REFS}"
-			(at 132.8216 21.59 0)
-			(hide yes)
-			(show_name no)
-			(do_not_autoplace no)
-			(effects
-				(font
-					(size 1.27 1.27)
-				)
-				(justify right)
-			)
-		)
-	)
 	(global_label "0_LED_C8"
 		(shape bidirectional)
@@
 		)
 	)
+	(global_label "0_FPGA_INITN"
+		(shape bidirectional)
+		(at 30.48 142.24 180)
+		(fields_autoplaced yes)
+		(effects
+			(font
+				(size 1.27 1.27)
+			)
+			(justify right)
+		)
+		(property "Intersheetrefs" "${INTERSHEET_REFS}"
+			(at 13.6834 142.24 0)
+			(hide yes)
+			(show_name no)
+			(do_not_autoplace no)
+			(effects
+				(font
+					(size 1.27 1.27)
+				)
+				(justify right)
+			)
+		)
+	)
 	(global_label "1_LED3"
 		(shape bidirectional)
@@
 			(hide yes)
 			(show_name no)
-			(do_not_autoplace no)
-			(effects
-				(font
-					(size 1.27 1.27)
-				)
-				(justify right)
-			)
-		)
-	)
-	(global_label "0_FPGA_INITN"
-		(shape bidirectional)
-		(at 149.86 19.05 180)
-		(fields_autoplaced yes)
-		(effects
-			(font
-				(size 1.27 1.27)
-			)
-			(justify right)
-		)
-		(property "Intersheetrefs" "${INTERSHEET_REFS}"
-			(at 133.0634 19.05 0)
-			(hide yes)
-			(show_name no)
