File: SIGMAGE_HW/SIGMAGE/DAC.kicad_sch (KiCad schematic)
At the start: 80 parts, among them J20 SJ63073E, J21 SJ63073E, J24 SJ63073E, J25 SJ63073E, U10 PCM5102APWR, U20 PCM5102APWR, U21 PCM5102APWR, U3 PCM5102APWR

Commit message: some foo
Changed lines of the file:
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@@
 		)
 		(property "Value" "1u"
-			(at 396.24 138.684 90)
+			(at 395.986 139.7 90)
 			(show_name no)
 			(do_not_autoplace no)

Commit message: improvements
Parts:
- C165, C166, C167, C168, C62, C63, C82, C83: footprint Resistor_SMD:R_0603_1608Metric -> Capacitor_SMD:C_0603_1608Metric
Connections:
- net 0_DAC1_DEMP is gone; now on net GND: U3.10 (DEMP)
- net 0_DAC1_FMT is gone; now on net GND: U3.16 (FMT)
- net 0_DAC2_CK is gone; now on net 0_BUS_DAC_BCK: U10.13 (BCK)
- net 0_DAC2_DEMP is gone; now on net GND: U10.10 (DEMP)
- net 0_DAC2_FMT is gone; now on net GND: U10.16 (FMT)
- net 0_DAC2_SCK is gone; now on net 0_BUS_DAC_SCK: U10.12 (SCK)
- net 0_DAC2_WS is gone; now on net 0_BUS_DAC_LRCK: U10.15 (LRCK)
- net 0_DAC3_CK is gone; now on net 0_BUS_DAC_BCK: U20.13 (BCK)
- net 0_DAC3_DEMP is gone; now on net GND: U20.10 (DEMP)
- net 0_DAC3_FMT is gone; now on net GND: U20.16 (FMT)
- net 0_DAC3_SCK is gone; now on net 0_BUS_DAC_SCK: U20.12 (SCK)
- net 0_DAC3_WS is gone; now on net 0_BUS_DAC_LRCK: U20.15 (LRCK)
- net 0_DAC4_CK is gone; now on net 0_BUS_DAC_BCK: U21.13 (BCK)
- net 0_DAC4_DEMP is gone; now on net GND: U21.10 (DEMP)
- net 0_DAC4_FMT is gone; now on net GND: U21.16 (FMT)
- net 0_DAC4_SCK is gone; now on net 0_BUS_DAC_SCK: U21.12 (SCK)
- net 0_DAC4_WS is gone; now on net 0_BUS_DAC_LRCK: U21.15 (LRCK)
- net 0_DAC1_CK renamed 0_BUS_DAC_BCK
- net 0_DAC1_SCK renamed 0_BUS_DAC_SCK
- net 0_DAC1_SD renamed 0_DAC1_DIN
- net 0_DAC1_WS renamed 0_BUS_DAC_LRCK
- net 0_DAC2_SD renamed 0_DAC2_DIN
- net 0_DAC3_SD renamed 0_DAC3_DIN
- net 0_DAC4_SD renamed 0_DAC4_DIN
Other:
- moved on the sheet: C145, C146, C147, C148, C149, C150, C151, C152, C153, C154, C155, C156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
