File: SIGMAGE_HW/SIGMAGE/FPGA.kicad_sch (KiCad schematic)
At the start: 52 parts, among them J9 TSW10607GS, U41 MMBT2222A, U8 LFE5U25F6BG256I

Commit message: changes
Connections:
- net DVCC_3V3: now also J9.1
- net FPGA_USART1_RX: now also J9.3; no longer J9.2, U8.T6 (PB4A)
- net FPGA_USART1_TX: now also J9.2; no longer J9.1, U8.R7 (PB6A)
- no-connect marks 3 -> 2

Commit message: finished schematic
Connections:
- net FPGA_CFG0 renamed 0_FPGA_CFG0
- net FPGA_CFG1 renamed 0_FPGA_CFG1
- net FPGA_CFG2 renamed 0_FPGA_CFG2
- net FPGA_DONE renamed 0_FPGA_DONE
- net FPGA_HOLDN renamed 0_FPGA_HOLDN
- net FPGA_INITN renamed 0_FPGA_INITN
- net FPGA_JTAG_TCK renamed 0_FPGA_JTAG_TCK
- net FPGA_JTAG_TDI renamed 0_FPGA_JTAG_TDI
- net FPGA_JTAG_TDO renamed 0_FPGA_JTAG_TDO
- net FPGA_JTAG_TMS renamed 0_FPGA_JTAG_TMS
- net FPGA_PROGRAMN renamed 0_FPGA_PROGRAMN
- net FPGA_SPI_CLK renamed 0_FPGA_SPI_CLK
- net FPGA_SPI_CS renamed 0_FPGA_SPI_CS
- net FPGA_SPI_MISO renamed 0_FPGA_SPI_MISO
- net FPGA_SPI_MOSI renamed 0_FPGA_SPI_MOSI
- net FPGA_USART1_RX renamed 0_FPGA_USART1_RX
- net FPGA_USART1_TX renamed 0_FPGA_USART1_TX
Other:
- moved on the sheet: R113, R114, R115, R116

Commit message: almost done with tha top part
Connections:
- net 0_FPGA_DONE: no longer R110.1
- net 0_FPGA_INITN: no longer D262.1 (K)
- new net 1_FPGA_DONE: R110.1
- new net 1_FPGA_INITN: D262.1 (K)

Commit message: some foo
Connections:
- net 0_LED_C2: now also U8.M9 (PB18A)
- net 0_LED_R15: now also U8.P8 (PB13B)
Changed lines of the file:
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@@
 		)
 	)
+	(global_label "0_LED_R15"
+		(shape bidirectional)
+		(at 369.57 50.8 0)
+		(fields_autoplaced yes)
+		(effects
+			(font
+				(size 1.27 1.27)
+			)
+			(justify left)
+		)
+		(property "Intersheetrefs" "${INTERSHEET_REFS}"
+			(at 383.9473 50.8 0)
+			(hide yes)
+			(show_name no)
+			(do_not_autoplace no)
+			(effects
+				(font
+					(size 1.27 1.27)
+				)
+				(justify left)
+			)
+		)
+	)
 	(global_label "0_ICOM_AUX3"
 		(shape bidirectional)
@@
 			(hide yes)
 			(show_name no)
+			(do_not_autoplace no)
+			(effects
+				(font
+					(size 1.27 1.27)
+				)
+				(justify left)
+			)
+		)
+	)
+	(global_label "0_LED_C2"
+		(shape bidirectional)
+		(at 369.57 45.72 0)
+		(fields_autoplaced yes)
+		(effects
+			(font
+				(size 1.27 1.27)
+			)
+			(justify left)
+		)
+		(property "Intersheetrefs" "${INTERSHEET_REFS}"
+			(at 382.7378 45.72 0)
+			(hide yes)
+			(show_name no)

Commit message: more foo
Connections:
- net 0_LED_C1: now also U8.B8 (PT35B)
- net 0_LED_C10: now also U8.A4 (PT6B)
- net 0_LED_C11: now also U8.B3 (PT4B)
- net 0_LED_C12: now also U8.A3 (PT6A)
- net 0_LED_C13: now also U8.B2 (PL2B)
- net 0_LED_C14: now also U8.A2 (PT4A)
- net 0_LED_C15: now also U8.C2 (PL5B)
- net 0_LED_C16: now also U8.B1 (PL2A)
- net 0_LED_C2: now also U8.A8 (PT29B); no longer U8.M9 (PB18A)
- net 0_LED_C3: now also U8.B7 (PT27B)
- net 0_LED_C4: now also U8.A7 (PT29A)
- net 0_LED_C5: now also U8.B6 (PT22B)
- net 0_LED_C6: now also U8.A6 (PT18B)
- net 0_LED_C7: now also U8.B5 (PT15B)
- net 0_LED_C8: now also U8.A5 (PT18A)
- net 0_LED_C9: now also U8.B4 (PT11B)
- net 0_LED_R1: now also U8.B16 (PR2A)
- net 0_LED_R10: now also U8.B12 (PT56A)
- net 0_LED_R11: now also U8.A11 (PT53A)
- net 0_LED_R12: now also U8.B11 (PT49A)
- net 0_LED_R13: now also U8.A10 (PT42B)
- net 0_LED_R14: now also U8.B10 (PT44A)
- net 0_LED_R15: now also U8.A9 (PT42A); no longer U8.P8 (PB13B)
- net 0_LED_R16: now also U8.B9 (PT38A)
- net 0_LED_R2: now also U8.C15 (PR5B)
- net 0_LED_R3: now also U8.A15 (PT67B)
- net 0_LED_R4: now also U8.B15 (PR2B)
- net 0_LED_R5: now also U8.A14 (PT65B)
- net 0_LED_R6: now also U8.B14 (PT67A)
- net 0_LED_R7: now also U8.A13 (PT65A)
- net 0_LED_R8: now also U8.B13 (PT60A)
- net 0_LED_R9: now also U8.A12 (PT53B)

Commit message: improvements
Parts:
- added R186, R187, R188, R189, R190, R191: 33, Resistor_SMD:R_0603_1608Metric, symbol Device:R
Connections:
- net 0_ADC1_DOUT: now also U8.M15 (PR26D)
- net 0_ADC1_OSR: now also U8.M16 (PR26C)
- net 0_ADC1_PDWN: now also U8.P16 (PR35A)
- net 0_ADC1_PYPAS: now also U8.N16 (PR32A)
- net 0_ADC2_DOUT: now also U8.K15 (PR23D)
- net 0_ADC2_OSR: now also U8.K16 (PR23C)
- net 0_ADC2_PDWN: now also U8.L15 (PR26B)
- net 0_ADC2_PYPAS: now also U8.L16 (PR26A)
- net 0_ADC3_DOUT: now also U8.F16 (PR14A)
- net 0_ADC3_OSR: now also U8.F15 (PR11C)
- net 0_ADC3_PDWN: now also U8.G16 (PR20A)
- net 0_ADC3_PYPAS: now also U8.G15 (PR14B)
- net 0_ADC4_DOUT: now also U8.D16 (PR8A)
- net 0_ADC4_OSR: now also U8.C16 (PR5A)
- net 0_ADC4_PDWN: now also U8.E16 (PR11D)
- net 0_ADC4_PYPAS: now also U8.E15 (PR8B)
- net 0_DAC_SCK: now reaches U8.H2 (PL20B)
- net 0_DAC_SCK: now also R189.2
- net 0_DAC_BCK: now reaches U8.J1 (PL23A)
- net 0_DAC_BCK: now also R190.2
- net 0_DAC_LRCK: now reaches U8.J2 (PL23B)
- net 0_DAC_LRCK: now also R191.2
- net 0_ADC_SCK: now reaches U8.H15 (PR20B)
- net 0_ADC_SCK: now also R186.2
- net 0_ADC_LRCK: now reaches U8.J15 (PR23B)
- net 0_ADC_LRCK: now also R188.2
- net 0_ADC_BCK: now reaches U8.J16 (PR23A)
- net 0_ADC_BCK: now also R187.2
- new net 0_BUS_ADC_BCK: R187.1
- new net 0_BUS_ADC_LRCK: R188.1
- new net 0_BUS_ADC_SCK: R186.1
- new net 0_BUS_DAC_BCK: R190.1
- new net 0_BUS_DAC_LRCK: R191.1
- new net 0_BUS_DAC_SCK: R189.1
